File: Ember_pilot_version/Ember_pilot_version.kicad_sch (KiCad schematic)
At the start: 18 parts, among them U2 BNO055, U4 BMP280

Commit message: gnss added
Parts:
- added C1: 10 uF, microbuilder:0603, symbol microbuilder:CAP_CERAMIC0603
- added C2, C3, C4: 120 pF, microbuilder:0603, symbol microbuilder:CAP_CERAMIC0603
- added FL1: ~, AFS14A04-1575.42-T3:FIL_AFS14A04-1575.42-T3, symbol AFS14A04-1575.42-T3:AFS14A04-1575.42-T3
- added J1: ~, sma-connector:RFSOLUTIONS_CON-SMA-EDGE-S, symbol sma-connector:CON-SMA-EDGE-S
- added L1: ~, inductor_0603:INDC1608X95N, symbol inductor_0603:LQM18PZ2R2MFHD
- added R1, R2: 10k ohm, adafruit:R0603, symbol adafruit:R-US_R0603
- added U6: ~, TESEO-LIV3F:TESEO-LIV3F, symbol TESEO-LIV3F:TESEO-LIV3F
Connections:
- net 3v3: now also C1.2 (P$2), R1.1, R2.1, U6.6 (VBATT), U6.7 (VCC_IO), U6.8 (VCC)
- net 5v: now also L1.1
- net GND: now also C1.1 (P$1), C4.1 (P$1), FL1.B (GND), FL1.D (GND), FL1.E (GND), J1.G1 (2), J1.G2 (2), J1.G3 (2), J1.G4 (2), U6.1 (GND), U6.10 (GND_RF), U6.12 (GND_RF)
- net GPS_TX: now reaches U1.GP11
- net GPS_TX: now also R2.2, U6.2 (TX)
- net GPS_RX: now reaches U1.GP12
- net GPS_RX: now also R1.2, U6.3 (RX)
- new net: C3.1 (P$1), C4.2 (P$2), J1.1, L1.2
- new net: C3.2 (P$2), FL1.C (IN)
- new net: C2.1 (P$1), FL1.A (OUT)
- new net: C2.2 (P$2), U6.11 (RF_IN)
Other:
- note added: "GNSS"

Commit message: LoRa, Buck converter and pyro (partially) added
Parts:
- added Buck_converter1: 4.7uH, SRN6045-4R7Y:SRN6045, symbol SRN6045-4R7Y:SRN6045-330M6045
- added C17: 3.3pF, microbuilder:0603, symbol microbuilder:CAP_CERAMIC0603
- added C18, C19, C22: 100nF, microbuilder:0603, symbol microbuilder:CAP_CERAMIC0603
- added C20, C21, C23: 22uF, microbuilder:0603, symbol microbuilder:CAP_CERAMIC0603
- added IC2: MP2315S, MP2315SGJ-Z:SOT65P280X100-8N, symbol MP2315SGJ-Z:MP2315SGJ-Z
- added J2: ~, sma-connector:RFSOLUTIONS_CON-SMA-EDGE-S, symbol sma-connector:CON-SMA-EDGE-S
- added J4: BATT_CONN, XT60-M:AMASS_XT60-M, symbol XT60-M:XT60-M
- added R10: 40.2k, adafruit:R0603, symbol adafruit:R-US_R0603
- added R11: 7.5k, adafruit:R0603, symbol adafruit:R-US_R0603
- added R12: 20k, adafruit:R0603, symbol adafruit:R-US_R0603
- added R13, R16, R18, R4: 33k, microbuilder:0603, symbol microbuilder:RESISTOR0603
- added R14, R17, R25, R5: 1k, microbuilder:0603, symbol microbuilder:RESISTOR0603
- added R6: 499k, adafruit:R0603, symbol adafruit:R-US_R0603
- added R7: 10, adafruit:R0603, symbol adafruit:R-US_R0603
- added R8: 100k, adafruit:R0603, symbol adafruit:R-US_R0603
- added R9: 9.09k, adafruit:R0603, symbol adafruit:R-US_R0603
- added U7 (x2), U8, U9: CJ3400, FLYTE_3.02:SOT91P240X120-3N, symbol FLYTE_3.02-eagle-import:BS170F_BS170F
- added X1: 22-23-2121, FLYTE_3.02:22-23-2121, symbol FLYTE_3.02-eagle-import:con-molex_165_22-23-2121
- FL1: value ~ -> Saw_filter
- U6: value ~ -> Teseo_liv3f
Connections:
- net 3v3: now also U5.8 (3V3), Buck_converter1.1, C20.2 (P$2), C21.2 (P$2)
- net 5v: now also C17.2 (P$2), R10.2
- net GND: now also U5.1 (GND), U5.15 (GND), U5.2 (GND), U5.7 (GND), C19.1 (P$1), C20.1 (P$1), C21.1 (P$1), C22.1 (P$1), C23.1 (P$1), IC2.4 (GND), J2.G1 (2), J2.G2 (2), J2.G3 (2), J2.G4 (2), J4.N (NEG), R11.1, R13.2, R16.2, R25.1, R4.2, R9.1, U7.2 (S), U7.2 (S), U9.2 (S), X1.12 (S)
- net GPS_RX: now also U1.GP4; no longer U1.GP12
- net GPS_TX: now also U1.GP5; no longer U1.GP11
- net SCL: now also U1.GP21; no longer U1.GP5
- net SDA: now also U1.GP20; no longer U1.GP4
- net LORA_RESET: now reaches U5.10 (RESET)
- net LORA_RESET: now also U1.GP12
- net LORA_MISO: now reaches U5.11 (MISO)
- net LORA_MISO: now also U1.GP8
- net LORA_MOSI: now reaches U5.12 (MOSI)
- net LORA_MOSI: now also U1.GP15
- net LORA_SCLK: now reaches U5.13 (CLK)
- net LORA_SCLK: now also U1.GP14
- net LORA_CS: now reaches U5.14 (CS)
- net LORA_CS: now also U1.GP13
- net at U5.16 (ANT): now also J2.1
- net LORA_DIO1: now reaches U5.6 (DIO1)
- net LORA_DIO1: now also U1.GP11
- net LORA_BUSY: now reaches U5.9 (BUSY)
- net LORA_BUSY: now also U1.GP9
- new net: R18.1, R25.2, U8.1 (G)
- new net: IC2.1 (AAM), R8.1, R9.2
- new net: R13.1, R14.2, U7.1 (G)
- new net: R4.1, R5.2, U9.1 (G)
- new net: R16.1, R17.2, U7.1 (G)
- new net: C18.1 (P$1), R7.2
- new net: IC2.5 (BST), R7.1
- new net: C17.1 (P$1), R10.1, R11.2, R12.1
- new net: IC2.8 (FB), R12.2
- new net: IC2.6 (EN), R6.1
- new net BC: X1.11 (S)
- new net BST: Buck_converter1.2, C18.2 (P$2), IC2.3 (SW)
- new net DROGUE: R14.1
- new net IGN1: R18.2, U8.2 (S)
- new net IGN2: R5.1
- new net MAIN: R17.1
- new net MOS: X1.10 (S)
- new net PYRO_DROGUE: U7.3 (D), X1.2 (S)
- new net PYRO_DROGUE2: U9.3 (D), X1.8 (S)
- new net PYRO_MAIN: U7.3 (D), X1.4 (S)
- new net PYRO_MAIN2: U8.3 (D), X1.6 (S)
- new net VCC_PYRO: X1.1 (S), X1.3 (S), X1.5 (S), X1.7 (S), X1.9 (S)
- new net V_BATT: C22.2 (P$2), C23.2 (P$2), IC2.2 (IN), J4.P (POS), R6.2
- new net V_CC_AAM: C19.2 (P$2), IC2.7 (VCC), R8.2
Other:
- note added: "Power Supply"
- moved on the sheet: U5

Commit message: Added Final Iterations in pilot version
Parts:
- added D1: ~, 0603_LED:0603.LED, symbol 0603_LED:LED.0603
- added LS1: BUZZER, CMT-8530S-SMT:CUI_CMT-8530S-SMT, symbol CMT-8530S-SMT:CMT-8530S-SMT
- added R15: 10 k, microbuilder:0603, symbol microbuilder:RESISTOR0603
- added R26, R3: 100 ohm, microbuilder:0603, symbol microbuilder:RESISTOR0603
- added U10: CJ3400, FLYTE_3.02:SOT91P240X120-3N, symbol FLYTE_3.02-eagle-import:BS170F_BS170F
Connections:
- net 3v3: now also U10.3 (D)
- net GND: now also R26.2
- net LED: now reaches U1.GP0
- net LED: now also D1.P$1 (1)
- net BUZZER: now reaches U1.GP1
- net BUZZER: now also R15.1, R3.2
- new net: LS1.N, R3.1
- new net: R15.2, U10.1 (G)
- new net: LS1.P, U10.2 (S)
- new net: D1.P$2 (2), R26.1
Other:
- note added: "BUZZER"
- moved on the sheet: R13, R14, R16, R17, R18, R25, R4, R5, U7, U8, X1A, X1B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

Commit message: changed buzzer circuit, pyro mosfets and finalized connections
Parts:
- removed R16, R18: 33k, microbuilder:0603, symbol microbuilder:RESISTOR0603
- removed R17, R25: 1k, microbuilder:0603, symbol microbuilder:RESISTOR0603
- removed U7 (x2), U8, U9: CJ3400, FLYTE_3.02:SOT91P240X120-3N, symbol FLYTE_3.02-eagle-import:BS170F_BS170F
- removed unit 3 of X1
- removed unit 4 of X1
- added D2: RSX501LAM20TR, RSX501LAM20TR:DIOM4725X105N, symbol RSX501LAM20TR:RSX501LAM20TR
- added Q1, Q2, Q3, Q4: SISA96DN-T1, SISA96DN-T1-GE3:SIS862DNT1GE3, symbol SISA96DN-T1-GE3:SISA96DN-T1-GE3
- added R27, R29, R31, R33: 1k, microbuilder:0603, symbol microbuilder:RESISTOR0603
- added R28, R30, R32: 33k, microbuilder:0603, symbol microbuilder:RESISTOR0603
- R13: value 33k -> 33K
- R14: value 1k -> 1K
- R15: value 10 k -> 100
- R3: value 100 ohm -> 33k
- U5: value ~ -> Waveshare_SX1262
Connections:
- net IGN2 is gone; now on net DROGUE2: R5.1
- net MOS is gone; now on net V_BATT: X1.10 (S)
- net 3v3: no longer U10.3 (D)
- net BUZZER: now also R27.1; no longer R15.1, R3.2
- net DROGUE: now also U1.GP6, R31.1; no longer R14.1
- net GND: now also LS1.N, R13.1, R3.2, Q1.1 (S_1), Q1.2 (S_2), Q1.3 (S_3), Q2.1 (S_1), Q2.2 (S_2), Q2.3 (S_3), Q3.1 (S_1), Q3.2 (S_2), Q3.3 (S_3), Q4.1 (S_1), Q4.2 (S_2), Q4.3 (S_3), R28.2, R30.2, R32.2; no longer R13.2
- net LED: now also U1.GP10; no longer U1.GP0
- net MAIN: now also U1.GP16, R33.1
- net PYRO_DROGUE: now also Q2.10 (D_6), Q2.11 (D_7), Q2.5 (D_1), Q2.6 (D_2), Q2.7 (D_3), Q2.8 (D_4), Q2.9 (D_5)
- net PYRO_DROGUE2: now also Q4.10 (D_6), Q4.11 (D_7), Q4.5 (D_1), Q4.6 (D_2), Q4.7 (D_3), Q4.8 (D_4), Q4.9 (D_5)
- net PYRO_MAIN: now also Q3.10 (D_6), Q3.11 (D_7), Q3.5 (D_1), Q3.6 (D_2), Q3.7 (D_3), Q3.8 (D_4), Q3.9 (D_5)
- net PYRO_MAIN2: now also Q1.10 (D_6), Q1.11 (D_7), Q1.5 (D_1), Q1.6 (D_2), Q1.7 (D_3), Q1.8 (D_4), Q1.9 (D_5)
- net VCC_PYRO: now also R14.2
- net V_BATT: no longer J4.P (POS)
- net at R3.1: now also U10.1 (G), R27.2; no longer LS1.N
- net at R4.1, R5.2: now also Q4.4 (G)
- net at R15.2: now also U10.3 (D); no longer U10.1 (G)
- net MAIN2: now reaches U1.GP17
- net MAIN2: now also R29.1
- net at U1.GP26_A0: now also R13.2, R14.1
- net DROGUE2: now reaches U1.GP7
- new net: Q3.4 (G), R32.1, R33.2
- new net: Q2.4 (G), R30.1, R31.2
- new net: Q1.4 (G), R28.1, R29.2
- new net: D2.2, J4.P (POS)
Other:
- note added: "BUZZER and LED"
- note removed: "BUZZER"
- moved on the sheet: Buck_converter1, C13, C14, C15, C16, C17, C18, C19, C20, C21, C22, C23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

Commit message: completed
Parts:
- added R16: ~, microbuilder:0603, symbol microbuilder:RESISTOR0603
- C13, C14, C15: value 10 uF -> 100 nF
- R13: value 33K -> 10k
- R14: value 1K -> 13k
Connections:
- net GND: now also R16.1
- net LORA_CS: now also R16.2
Changed lines of the file:
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@@
 	)
 	(junction
+		(at 266.7 73.66)
+		(diameter 0)
+		(color 0 0 0 0)
+	)
+	(junction
 		(at 374.65 331.47)
 		(diameter 0)
@@
 	(wire
 		(pts
+			(xy 266.7 73.66) (xy 266.7 74.93)
+		)
+		(stroke
+			(width 0)
+			(type default)
+		)
+	)
+	(wire
+		(pts
 			(xy 414.02 342.9) (xy 420.37 342.9)
 		)
@@
 	(wire
 		(pts
+			(xy 266.7 73.66) (xy 285.75 73.66)
+		)
+		(stroke
+			(width 0)
+			(type default)
+		)
+	)
+	(wire
+		(pts
 			(xy 496.57 62.23) (xy 496.57 66.04)
 		)
@@
 	(wire
 		(pts
-			(xy 280.67 73.66) (xy 285.75 73.66)
-		)
-		(stroke
-			(width 0)
-			(type default)
-		)
-	)
-	(wire
-		(pts
 			(xy 85.09 231.14) (xy 85.09 232.41)
 		)
@@
 	(wire
 		(pts
+			(xy 266.7 69.85) (xy 266.7 73.66)
+		)
+		(stroke
+			(width 0)
+			(type default)
+		)
+	)
+	(wire
+		(pts
 			(xy 482.6 77.47) (xy 486.41 77.47)
 		)
@@
 	(wire
 		(pts
+			(xy 266.7 85.09) (xy 266.7 90.17)
+		)
+		(stroke
+			(width 0)
+			(type default)
+		)
+	)
+	(wire
+		(pts
 			(xy 59.69 266.7) (xy 59.69 269.24)
 		)
@@
 	)
 	(label "GND"
+		(at 266.7 90.17 0)
+		(effects
+			(font
+				(size 1.27 1.27)
+			)
+			(justify left bottom)
+		)
+	)
+	(label "GND"
 		(at 496.57 74.93 0)
 		(effects
@@
 	)
 	(label "LORA_CS"
-		(at 280.67 73.66 180)
+		(at 266.7 69.85 180)
 		(effects
 			(font
@@
 			)
 		)
-		(property "Value" "10 uF"
+		(property "Value" "100 nF"
 			(at 491.49 196.85 90)
 			(effects
@@
 			)
 		)
-		(property "Value" "10 uF"
+		(property "Value" "100 nF"
 			(at 501.65 40.64 90)
 			(effects
@@
 			)
 		)
-		(property "Value" "10 uF"
+		(property "Value" "100 nF"
 			(at 525.78 137.16 90)
 			(effects
@@
 			)
 		)
-		(property "Value" "33K"
+		(property "Value" "10k"
 			(at 289.56 298.4499 90)
 			(effects
@@
 			)
 		)
-		(property "Value" "1K"
+		(property "Value" "13k"
 			(at 293.37 287.02 0)
 			(effects
@@
 				)
 			)
+		)
+	)
+	(symbol
+		(lib_id "microbuilder:RESISTOR0603")
+		(at 266.7 80.01 90)
+		(unit 1)
+		(exclude_from_sim no)
+		(in_bom yes)
+		(on_board yes)
+		(dnp no)
+		(fields_autoplaced yes)
+		(property "Reference" "R16"
+			(at 269.24 78.7399 90)
+			(effects
+				(font
+					(size 1.27 1.27)
+				)
+				(justify right)
+			)
+		)
+		(property "Value" "~"
+			(at 269.24 81.2799 90)
+			(effects
+				(font
+					(size 1.27 1.27)
+				)
+				(justify right)
+			)
+		)
+		(property "Footprint" "microbuilder:0603"
+			(at 266.7 80.01 0)
+			(effects
+				(font
+					(size 1.27 1.27)
+				)
+				(hide yes)
+			)
+		)
+		(property "Datasheet" ""
+			(at 266.7 80.01 0)
+			(effects
+				(font
+					(size 1.27 1.27)
+				)
+				(hide yes)
+			)
+		)
+		(property "Description" "Resistors\n\n0402 - 0402 Surface Mount Package\n\n• 22 Ohm 1% 1/16W [Digikey: 311-22.0LRTR-ND]\n• 33 Ohm 5% 1/16W\n• 1.0K 5% 1/16W\n• 1.5K 5% 1/16W\n• 2.0K 1% 1/16W\n• 10.0K 1% 1/16W [Digikey: 311-10.0KLRTR-ND]\n• 10.0K 5% 1/16W [Digikey: RMCF0402JT10K0TR-ND]\n• 12.1K 1% 1/16W [Digikey: 311-22.0LRTR-ND]\n• 100.0K 5% 1/16W\n\n0603 - 0603 Surface Mount Package\n\n• 0 Ohm 1/10 Watt 1% Resistor\n• 15 Ohm 1/10 Watt 1% Resistor\n• 33 Ohm 1/10 Watt 1% Resistor\n• 49.9 Ohm 1/10 Watt 1% Resistor\n• 100 Ohm 1/10 Watt 1% Resistor\n• 150 Ohm 1/10 Watt 1% Resistor\n• 240 Ohm 1/10 Watt 1% Resistor\n• 390 Ohm 1/10 Watt 1% Resistor\n• 560 Ohm 1/10 Watt 1% Resistor\n• 680 Ohm 1/10 Watt 1% Resistor\n• 750 Ohm 1/10 Watt 1% Resistor\n• 1.0K Ohm 1/10 Watt 1% Resistor\n• 1.5K Ohm 1/10 Watt 1% Resistor\n• 2.0K Ohm 1/10 Watt 1% Resistor\n• 2.2K Ohm 1/10 Watt 1% Resistor\n• 3.3K Ohm 1/10 Watt 1% Resistor\n• 4.7K Ohm 1/10 Watt 1% Resistor\n• 10.0K Ohm 1/10 Watt 1% Resistor\n• 12.0K Ohm 1/10 Watt 1% Resistor\n• 12.1K Ohm 1/10 Watt 1% Resistor\n• 20.0K Ohm 1/10 Watt 1% Resistor\n• 33.0K Ohm 1/10 Watt 1% Resistor\n• 100.0K Ohm 1/10 Watt 1% Resistor\n\n0805 - 0805 Surface Mount Package\n\n• 0 Ohm 1/8 Watt 1% Resistor\n• 33 Ohm 1/8 Watt 1% Resistor\n• 100 Ohm 1/8 Watt 1% Resistor\n• 150 Ohm 1/8 Watt 1% Resistor\n• 200 Ohm 1/8 Watt 1% Resistor\n• 240 Ohm 1/8 Watt 1% Resistor\n• 330 Ohm 1/8 Watt 1% Resistor\n• 390 Ohm 1/8 Watt 1% Resistor\n• 470 Ohm 1/8 Watt 1% Resistor\n• 1.0K Ohm 1/8 Watt 1% Resistor\n• 1.5K Ohm 1/8 Watt 1% Resistor\n• 2.0K Ohm 1/8 Watt 1% Resistor\n• 4.7K Ohm 1/8 Watt 1% Resistor\n• 5.1K Ohm 1/8 Watt 1% Resistor\n• 5.6K Ohm 1/8 Watt 1% Resistor\n• 10.0K Ohm 1/8 Watt 1% Resistor\n• 22.0K Ohm 1/8 Watt 1% Resistor\n• 33.0K Ohm 1/8 Watt 1% Resistor\n• 100K Ohm 1/8 Watt 1% Resistor\n\n1206 - 1206 Surface Mount Package  2012 - 2010 Surface Mount Package\n\n• 0.11 Ohm 1/2 Watt 1% Resistor - Digikey: RHM.11UCT-ND"
+			(at 266.7 80.01 0)
+			(effects
+				(font
+					(size 1.27 1.27)
+				)
+				(hide yes)
+			)
+		)
+		(pin "1"
+		)
+		(pin "2"
+		)
+		(instances
+			(project ""
+				(path "/3d6c902b-75d5-4305-b725-f5c596d25bec"
+					(reference "R16")
+					(unit 1)
+				)
+			)

Commit message: issues resolved
Parts:
- removed D1: ~, 0603_LED:0603.LED, symbol 0603_LED:LED.0603
- removed L1: ~, inductor_0603:INDC1608X95N, symbol inductor_0603:LQM18PZ2R2MFHD
- removed LS1: BUZZER, CMT-8530S-SMT:CUI_CMT-8530S-SMT, symbol CMT-8530S-SMT:CMT-8530S-SMT
- removed R26: 100 ohm, microbuilder:0603, symbol microbuilder:RESISTOR0603
- removed U10: CJ3400, FLYTE_3.02:SOT91P240X120-3N, symbol FLYTE_3.02-eagle-import:BS170F_BS170F
- removed X1: 22-23-2121, FLYTE_3.02:22-23-2121, symbol FLYTE_3.02-eagle-import:con-molex_165_22-23-2121
- added J3, J5, J6, J7, J8: ~, OSTTA020161:ONSHORE_OSTTA020161, symbol OSTTA020161:OSTTA020161
- added L2: ~, microbuilder:0603, symbol microbuilder:INDUCTOR0603
- added LED1: BATT_CONN, microbuilder:CHIPLED_0603, symbol microbuilder:LED0603
- added LS2: BUZZER, CMT-8530S-SMT:CUI_CMT-8530S-SMT, symbol CMT-8530S-SMT:CMT-8530S-SMT
- added Q5: CJ3400, CJ3400:SOT95P240X115-3N, symbol CJ3400:CJ3400
- added R17: 100, microbuilder:0603, symbol microbuilder:RESISTOR0603
Connections:
- net 3v3: now also R15.1
- net 5v: now also L2.1
- net GND: now also LS2.N, R17.1
- net PYRO_DROGUE: now also J3.2
- net PYRO_DROGUE2: now also J7.2
- net PYRO_MAIN: now also J5.2
- net PYRO_MAIN2: now also J6.2
- net VCC_PYRO: now also J3.1, J5.1, J6.1, J7.1, J8.1
- net V_BATT: now also D2.1, J8.2, LED1.A
- net at C3.1 (P$1), C4.2 (P$2), J1.1: now also L2.2
- net at R27.2, R3.1: now also Q5.1 (G)
- net at R15.2: now also Q5.3 (D)
- new net: LED1.C, R17.2
- new net: LS2.P, Q5.2 (S)
Other:
- note added: "BUZZER"
- note removed: "BUZZER and LED"

Commit message: routing started
Parts:
- removed U1: ~, RASPBERRY_PI_PICO:RASPBERRY_PI_PICO, symbol RASPBERRY_PI_PICO:RASPBERRY_PI_PICO
- added U7: ~, RpiPico:PICO-PKG-SMD, symbol RpiPico:RASPBERRY_PICOSMD
- J3: value ~ -> DROGUE
- J5: value ~ -> MAIN
- J6: value ~ -> MAN2
- J7: value ~ -> DROGUE2
- J8: value ~ -> ARM
- R16: value ~ -> 4.7k
Connections:
- net 3v3: now also Q5.3 (D), U7.P$36 (3V3(OUT)); no longer Buck_converter1.1, C20.2 (P$2), C21.2 (P$2), R15.1
- net 5v: now also Buck_converter1.1, C20.2 (P$2), C21.2 (P$2), U7.P$39 (VSYS)
- net BUZZER: now also U7.P$4 (GP2)
- net DROGUE: now also U7.P$9 (GP6)
- net DROGUE2: now also U7.P$10 (GP7)
- net GND: now also R15.2, U7.P$13 (GND), U7.P$18 (GND), U7.P$23 (GND), U7.P$28 (GND), U7.P$3 (GND), U7.P$33 (GND), U7.P$38 (GND), U7.P$8 (GND); no longer LS2.N
- net GPS_RX: now also U7.P$6 (GP4)
- net GPS_TX: now also U7.P$7 (GP5)
- net LORA_BUSY: now also U7.P$12 (GP9)
- net LORA_CS: now also U7.P$17 (GP13)
- net LORA_DIO1: now also U7.P$15 (GP11)
- net LORA_MISO: now also U7.P$11 (GP8)
- net LORA_MOSI: now also U7.P$20 (GP15)
- net LORA_RESET: now also U7.P$16 (GP12)
- net LORA_SCLK: now also U7.P$19 (GP14)
- net MAIN: now also U7.P$21 (GP16)
- net MAIN2: now also U7.P$22 (GP17)
- net SCL: now also U7.P$27 (GP21)
- net SDA: now also U7.P$26 (GP20)
- net AAM_DIV: now reaches IC2.1 (AAM), R8.1, R9.2
- net BST_INN: now reaches C18.1 (P$1), R7.2
- net BST_IN: now reaches IC2.5 (BST), R7.1
- net at R13.2, R14.1: now also U7.P$35 (ADC_REF)
- net V_DIV: now reaches C17.1 (P$1), R10.1, R11.2, R12.1
- net BATT_IN: now reaches D2.2, J4.P (POS)
- net FB_IN: now reaches IC2.8 (FB), R12.2
- net VCC_EN: now reaches IC2.6 (EN), R6.1
- net BST renamed FB
- new net: LS2.N, R15.1
Other:
- note added: "BMP280"
- note added: "BNO055"
- note added: "KX134"
- note added: "LORA"
- note removed: "BMP"
- note removed: "BNO"
- note removed: "KX"
- moved on the sheet: Buck_converter1, C1, C13, C14, C15, C16, C17, C18, C19, C2, C20, C21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

Commit message: initial layout done, rf traces remaining
Parts:
- removed Buck_converter1: 4.7uH, SRN6045-4R7Y:SRN6045, symbol SRN6045-4R7Y:SRN6045-330M6045
- removed C17: 3.3pF, microbuilder:0603, symbol microbuilder:CAP_CERAMIC0603
- removed C18, C19, C22: 100nF, microbuilder:0603, symbol microbuilder:CAP_CERAMIC0603
- removed C20, C21, C23: 22uF, microbuilder:0603, symbol microbuilder:CAP_CERAMIC0603
- removed IC2: MP2315S, MP2315SGJ-Z:SOT65P280X100-8N, symbol MP2315SGJ-Z:MP2315SGJ-Z
- removed R10: 40.2k, adafruit:R0603, symbol adafruit:R-US_R0603
- removed R11: 7.5k, adafruit:R0603, symbol adafruit:R-US_R0603
- removed R12: 20k, adafruit:R0603, symbol adafruit:R-US_R0603
- removed R6: 499k, adafruit:R0603, symbol adafruit:R-US_R0603
- removed R7: 10, adafruit:R0603, symbol adafruit:R-US_R0603
- removed R8: 100k, adafruit:R0603, symbol adafruit:R-US_R0603
- removed R9: 9.09k, adafruit:R0603, symbol adafruit:R-US_R0603
- added C5, C6, C7: 10 uF, microbuilder:0603, symbol microbuilder:CAP_CERAMIC0603
- added U1: LDO Regulator 5v, AMS1117-5.0:SOT229P700X180-4N, symbol AMS1117-5.0:AMS1117-5.0
Connections:
- net 5v: now also C6.1 (P$1), C7.1 (P$1), U1.2 (VOUT)
- net GND: now also C5.2 (P$2), C6.2 (P$2), C7.2 (P$2), U1.1 (GND/ADJ)
- net V_BATT: now also C5.1 (P$1), U1.3 (VIN)
- net G_MAIN: now reaches Q3.4 (G), R32.1, R33.2
- net G_DROGUE: now reaches Q2.4 (G), R30.1, R31.2
- net G_MAIN2: now reaches Q1.4 (G), R28.1, R29.2
