File: Ember_v1.0/Ember_v1.0.kicad_sch (KiCad schematic)
At the start: 12 parts

Commit message: Added power supply
Parts:
- added 1: 4.7uH, SRN6045-4R7Y:SRN6045, symbol SRN6045-4R7Y:SRN6045-330M6045
- added C17: 3.3pF, microbuilder:0603, symbol microbuilder:CAP_CERAMIC0603
- added C18, C19, C22: 100nF, microbuilder:0603, symbol microbuilder:CAP_CERAMIC0603
- added C20, C21, C23: 22uF, microbuilder:0603, symbol microbuilder:CAP_CERAMIC0603
- added D1, D2: RSX501LAM20TR, RSX501LAM20TR:DIOM4725X105N, symbol RSX501LAM20TR:RSX501LAM20TR
- added IC2: MP2315S, MP2315SGJ-Z:SOT65P280X100-8N, symbol MP2315SGJ-Z:MP2315SGJ-Z
- added J1: USB_C, USB4110GFA:GCT_USB4110GFA, symbol USB4110GFA:USB4110GFA
- added J2: BATT_CONN, XT60-M:AMASS_XT60-M, symbol XT60-M:XT60-M
- added LED1: V_BATT, adafruit:CHIP-LED0603, symbol adafruit:LEDCHIP-LED0603
- added LED2: VBUS, adafruit:CHIP-LED0603, symbol adafruit:LEDCHIP-LED0603
- added R10, R8: 100k, adafruit:R0603, symbol adafruit:R-US_R0603
- added R11: 31.6k, adafruit:R0603, symbol adafruit:R-US_R0603
- added R12: 20k, adafruit:R0603, symbol adafruit:R-US_R0603
- added R13, R14: 100, adafruit:R0603, symbol adafruit:R-US_R0603
- added R2, R3: 5.1k, adafruit:R0603, symbol adafruit:R-US_R0603
- added R4, R5: 27.4, adafruit:R0603, symbol adafruit:R-US_R0603
- added R6: 499k, adafruit:R0603, symbol adafruit:R-US_R0603
- added R7: 10, adafruit:R0603, symbol adafruit:R-US_R0603
- added R9: 9.09k, adafruit:R0603, symbol adafruit:R-US_R0603
Connections:
- net 3v3: now also 1.1, C17.2 (P$2), C20.2 (P$2), C21.2 (P$2), R10.2
- net GND: now also C19.1 (P$1), C20.1 (P$1), C21.1 (P$1), C22.1 (P$1), C23.1 (P$1), IC2.4 (GND), J1.A1/B12 (GND), J1.B1/A12 (GND), J1.S1 (GND), J1.S2 (GND), J1.S3 (GND), J1.S4 (GND), J2.N (NEG), R11.1, R13.2, R14.2, R2.2, R3.1, R9.1
- net D_M: now reaches IC1.66 (USB_DM)
- net D_M: now also R5.1
- net D_P: now reaches IC1.67 (USB_DP)
- net D_P: now also R4.1
- new net: IC2.1 (AAM), R8.1, R9.2
- new net: C18.1 (P$1), R7.2
- new net: IC2.5 (BST), R7.1
- new net: J1.A5 (CC1), R3.2
- new net: J1.A7 (DN1), R5.2
- new net: J1.A6 (DP1), R4.2
- new net: J1.B5 (CC2), R2.1
- new net: C17.1 (P$1), R10.1, R11.2, R12.1
- new net: LED1.C, R14.1
- new net: IC2.8 (FB), R12.2
- new net: IC2.6 (EN), R6.1
- new net: LED2.C, R13.1
- new net BST: 1.2, C18.2 (P$2), IC2.3 (SW)
- new net VBUS: D2.2, J1.A4/B9 (VBUS), J1.B4/A9 (VBUS), LED2.A
- new net V_BATT: D1.2, J2.P (POS), LED1.A
- new net V_CC_AAM: C19.2 (P$2), IC2.7 (VCC), R8.2
- new net V_MUX_OUT: C22.2 (P$2), C23.2 (P$2), D1.1, D2.1, IC2.2 (IN), R6.2
Other:
- note added: "Power Supply"
- moved on the sheet: C1, C2, C3, C4, C5, C6, C7, C8, C9, IC1, L1, R1

Commit message: Added the flash, XTAL remaining
Parts:
- added C10: 100nF, microbuilder:0603, symbol microbuilder:CAP_CERAMIC0603
- added R15: 10k, microbuilder:0603, symbol microbuilder:RESISTOR0603
- added R16: 0, microbuilder:0603, symbol microbuilder:RESISTOR0603
- added R17: ~, microbuilder:0603, symbol microbuilder:RESISTOR0603
- added S1: ~, DTS-3:DTS-3, symbol DTS-3:DTS-3
- added U1: FLASH_128K, W25Q32JVSSIQ:SOIC127P790X216-8N, symbol W25Q32JVSSIQ:W25Q32JVSSIQ
Connections:
- net 3v3: now also C10.1 (P$1), R15.2, U1.8 (VCC)
- net GND: now also C10.2 (P$2), S1.2, U1.4 (GND)
- net QSPI_SD3: now reaches IC1.70 (QSPI_SD3)
- net QSPI_SD3: now also U1.7 (~{HOLD}/~{RESET}(IO3))
- net QSPI_SCLK: now reaches IC1.71 (QSPI_SCLK)
- net QSPI_SCLK: now also U1.6 (CLK)
- net QSPI_SD0: now reaches IC1.72 (QSPI_SD0)
- net QSPI_SD0: now also U1.5 (DI(IO0))
- net QSPI_SD2: now reaches IC1.73 (QSPI_SD2)
- net QSPI_SD2: now also U1.3 (~{WP}(IO2))
- net QSPI_SD1: now reaches IC1.74 (QSPI_SD1)
- net QSPI_SD1: now also U1.2 (DO(IO1))
- net QSPI_SS: now reaches IC1.75 (QSPI_SS)
- net QSPI_SS: now also R17.2
- net FLASH_EXT_CS: now reaches IC1.77 (GPIO0)
- net FLASH_EXT_CS: now also R16.2
- new net: R17.1, S1.1
- new net: R15.1, R16.1, U1.1 (~{CS})
Other:
- note added: "External Flash"
- note added: "FLASH"
- note added: "Internal Flash Bootsel"

Commit message: Added xtal
Parts:
- added C11, C12: 18pF, microbuilder:0603, symbol microbuilder:CAP_CERAMIC0603
- added R18: 1k, microbuilder:0603, symbol microbuilder:RESISTOR0603
- added Y1: ~, YSX321SL:YSX321SL, symbol YSX321SL:YSX321SL
Connections:
- net GND: now also C11.2 (P$2), C12.1 (P$1), Y1.2 (GND_1), Y1.4 (GND_2)
- net XIN: now reaches IC1.30 (XIN)
- net XIN: now also C12.2 (P$2), Y1.3 (CRYSTAL_2)
- net XOUT: now reaches IC1.31 (XOUT)
- net XOUT: now also R18.1
- new net: C11.1 (P$1), R18.2, Y1.1 (CRYSTAL_1)
Other:
- note added: "Crystal Oscillator"

Commit message: Sensors done, some issues to be resolved
Parts:
- added C13, C14, C15: 10 uF, microbuilder:0603, symbol microbuilder:CAP_CERAMIC0603
- added C16: 100nF, microbuilder:0603, symbol microbuilder:CAP_CERAMIC0603
- added C24, C25: 27 pF, microbuilder:0603, symbol microbuilder:CAP_CERAMIC0603
- added R19, R20, R21, R22, R23, R24: 10k ohm, adafruit:R0603, symbol adafruit:R-US_R0603
- added U2: BNO055, Package_LGA:LGA-28_5.2x3.8mm_P0.5mm, symbol Sensor_Motion:BNO055
- added U3: ~, kx134:LGA12_2X2X0P9_ROM, symbol kx134:KX134-1211
- added U4: BMP280, Package_LGA:Bosch_LGA-8_2x2.5mm_P0.65mm_ClockwisePinNumbering, symbol Sensor_Pressure:BMP280
- added Y2: FC-135_32.7680KA-A0, XTAL_FC-135_32.7680KA-A0, symbol FC-135_32.7680KA-A0:FC-135_32.7680KA-A0
- renumbered 1 to 11111111
Connections:
- net 3v3: now also C13.2 (P$2), C14.1 (P$1), C15.1 (P$1), R20.1, R21.1, R22.1, R24.1, U2.28 (VDDIO), U2.3 (VDD), U2.4 (~{BOOT_LOAD_PIN}), U3.1 (SDO/ADDR), U3.10 (NCS), U3.3 (IO_VDD), U3.7 (VDD), U4.6 (VDDIO), U4.8 (VDD)
- net GND: now also C13.1 (P$1), C14.2 (P$2), C15.2 (P$2), C16.1 (P$1), C24.1 (P$1), C25.1 (P$1), R19.1, R23.1, U2.18 (COM2), U2.2 (GND), U2.25 (GNDIO), U2.5 (PS1), U2.6 (PS0), U3.4 (TRIG), U3.8 (GND_2), U3.9 (GND), U4.1 (GND), U4.7 (GND)
- net SDA: now reaches IC1.1 (GPIO4)
- net SDA: now also R20.2, U2.20 (COM0), U3.2 (SDI/SDA), U4.3 (SDI)
- net SCL: now reaches IC1.2 (GPIO5)
- net SCL: now also R21.2, U2.19 (COM1), U3.12 (SCLK/SCL), U4.4 (SCK)
- new net: R24.2, U4.2 (CSB)
- new net: R19.2, U4.5 (SDO)
- new net: R22.2, U2.11 (~{RESET})
- new net: R23.2, U2.17 (COM3)
- new net: C16.2 (P$2), U2.9 (CAP)
- new net XIN32: C24.2 (P$2), U2.27 (XIN32), Y2.1
- new net XOUT32: C25.2 (P$2), U2.26 (XOUT32), Y2.2
Other:
- note added: "BMP"
- note added: "BNO"
- note added: "KX"
- note added: "PULL UPS"

Commit message: crystal error resolved
Parts:
- removed Y2: FC-135_32.7680KA-A0, XTAL_FC-135_32.7680KA-A0, symbol FC-135_32.7680KA-A0:FC-135_32.7680KA-A0
- added XTAL1: XTAL_FC135, Q13FC1350000400:XTAL_FC-135_EPS, symbol Q13FC1350000400:Q13FC1350000400
- C24, C25: value 27 pF -> 20 pF
- renumbered 11111111 to Buck_converter1
Connections:
- net XIN32: now also XTAL1.1
- net XOUT32: now also XTAL1.2
Other:
- moved on the sheet: C25
Changed lines of the file:
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@@
 	)
 	(junction
-		(at 833.12 403.86)
-		(diameter 0)
-		(color 0 0 0 0)
-	)
-	(junction
 		(at 109.22 443.23)
 		(diameter 0)
@@
 	)
 	(junction
+		(at 822.96 403.86)
+		(diameter 0)
+		(color 0 0 0 0)
+	)
+	(junction
 		(at 142.24 433.07)
 		(diameter 0)
@@
 	(wire
 		(pts
-			(xy 833.12 403.86) (xy 833.12 410.21)
+			(xy 822.96 403.86) (xy 822.96 410.21)
 		)
 		(stroke
@@
 	(wire
 		(pts
-			(xy 833.12 417.83) (xy 833.12 420.37)
+			(xy 822.96 417.83) (xy 822.96 420.37)
 		)
 		(stroke
@@
 	(wire
 		(pts
-			(xy 833.12 403.86) (xy 838.2 403.86)
+			(xy 822.96 403.86) (xy 828.04 403.86)
 		)
 		(stroke
@@
 	(wire
 		(pts
-			(xy 829.31 403.86) (xy 833.12 403.86)
+			(xy 819.15 403.86) (xy 822.96 403.86)
 		)
 		(stroke
@@
 	)
 	(label "XOUT32"
-		(at 838.2 403.86 180)
+		(at 828.04 403.86 180)
 		(effects
 			(font
@@
 	)
 	(label "GND"
-		(at 833.12 420.37 0)
+		(at 822.96 420.37 0)
 		(effects
 			(font
@@
 		(dnp no)
 		(fields_autoplaced yes)
-		(property "Reference" "11111111"
+		(property "Reference" "Buck_converter1"
 			(at 167.64 452.12 0)
 			(effects
@@
 			(project ""
 				(path "/ce36a1c2-88cc-4cba-88a9-6235c3ec0ad6"
-					(reference "11111111")
+					(reference "Buck_converter1")
 					(unit 1)
 				)
@@
 	(symbol
 		(lib_id "microbuilder:CAP_CERAMIC0603")
-		(at 833.12 412.75 180)
+		(at 822.96 412.75 180)
 		(unit 1)
 		(exclude_from_sim no)
@@
 		(fields_autoplaced yes)
 		(property "Reference" "C25"
-			(at 835.66 412.7499 0)
+			(at 825.5 412.7499 0)
 			(effects
 				(font
@@
 			)
 		)
-		(property "Value" "27 pF"
-			(at 835.66 415.2899 0)
+		(property "Value" "20 pF"
+			(at 825.5 415.2899 0)
 			(effects
 				(font
@@
 		)
 		(property "Footprint" "microbuilder:0603"
-			(at 833.12 412.75 0)
+			(at 822.96 412.75 0)
 			(effects
 				(font
@@
 		)
 		(property "Datasheet" ""
-			(at 833.12 412.75 0)
+			(at 822.96 412.75 0)
 			(effects
 				(font
@@
 		)
 		(property "Description" "Ceramic Capacitors\n\n0402 - 0402 Surface Mount Capacitors\n\n• 16pF 50V 5% [Digikey: 445-4899-2-ND]\n• 18pF 50V 5% [Digikey: 490-1281-2-ND]\n• 22pF 50V 5% [Digikey: 490-1283-2-ND]\n• 68pF 50V 5% [Digikey: 490-1289-2-ND]\n• 0.1uF 10V 10% [Digikey: 490-1318-2-ND]\n• 1.0uF 6.3V 10% [Digikey: 490-1320-2-ND]\n\n0603 - 0603 Surface Mount Capacitors\n\n• 16 pF 50V 5% [Digikey: 445-5051-2-ND]\n• 22 pF 50V [Digikey: PCC220ACVTR-ND]\n• 33 pF 50V 5% [Digikey: 490-1415-1-ND]\n• 56pF 50V 5% [Digikey: 490-1421-1-ND]\n• 220pF 50V 5% [Digikey: 445-1285-1-ND]\n• 680 pF 50V\n• 2200 pF 50V 5% C0G [Digikey: 445-1297-1-ND]\n• 5600 pF 100V 5% X7R [Digikey: 478-3711-1-ND]\n• 0.1 µF 25V 10% [Digikey: PCC2277TR-ND]\n• 0.22 µF 16V 10% X7R [Digikey: 445-1318-1-ND]\n• 1.0 µF 25V 10% [Digikey: 445-5146-2-ND]\n\n0603 - RF Specific\n\n• 3pF 250V +/-0.1pF RF [Digikey: 712-1347-1-ND]\n• 18 pF 250V 5%  [Digikey: 478-3505-1-ND or 712-1322-1-ND]\n• 56 pF 250V 5% C0G RF [Digikey: 490-4867-1-ND]\n• 68 pF 250V RF [Digikey: 490-4868-1-ND]\n\n0805 - 0805 Surface Mount Capacitors\n\n• 220 pF 250V 2% RF Ceramic Capacitor [Digikey: 712-1398-1-ND]\n• 1000 pF 50V 2% NP0 Ceramic Capacitor [Digikey: 478-3760-1-ND]\n• 0.1 µF 25V 10% Ceramic Capacitor [Digikey: PCC1828TR-ND]\n• 1.0 µF 16V 10% Ceramic Capacitor[Digikey: 490-1691-2-ND]\n• 10.0 µF 10V 10% Ceramic Capacitor[Digikey: 709-1228-1-ND]\n• 10.0 uF 16V 10% Ceramic Capacitor [Digikey: 478-5165-2-ND]\n• 47 uF 6.3V 20% Ceramic Capacitor [Digikey: 587-1779-1-ND or 399-5506-1-ND]\n\n1206 - 1206 Surface Mount Capacitors\n\n• 47uF 10V 20% Ceramic Capacitor [Digikey: 490-5528-1-ND or 399-5508-1-ND or 445-6010-1-ND]\n• 100uF 6.3V -20%, +80% Y5V Ceramic Capacitor (Digikey: 490-4512-1-ND, Mouser: 81-GRM31CF50J107ZE1L)"
-			(at 833.12 412.75 0)
+			(at 822.96 412.75 0)
 			(effects
 				(font
@@
 	)
 	(symbol
+		(lib_id "Q13FC1350000400:Q13FC1350000400")
+		(at 808.99 403.86 0)
+		(unit 1)
+		(exclude_from_sim no)
+		(in_bom yes)
+		(on_board yes)
+		(dnp no)
+		(fields_autoplaced yes)
+		(property "Reference" "XTAL1"
+			(at 814.07 391.16 0)
+			(effects
+				(font
+					(size 3.4798 2.9578)
+				)
+			)
+		)
+		(property "Value" "XTAL_FC135"
+			(at 814.07 397.51 0)
+			(effects
+				(font
+					(size 3.4798 2.9578)
+				)
+			)
+		)
+		(property "Footprint" "Q13FC1350000400:XTAL_FC-135_EPS"
+			(at 808.99 403.86 0)
+			(effects
+				(font
+					(size 1.27 1.27)
+				)
+				(hide yes)
+			)
+		)
+		(property "Datasheet" ""
+			(at 808.99 403.86 0)
+			(effects
+				(font
+					(size 1.27 1.27)
+				)
+				(hide yes)
+			)
+		)
+		(property "Description" "https://pricing.snapeda.com/parts/Q13FC1350000400/EPSON/view-part?ref=eda Check availability"
+			(at 808.99 403.86 0)
+			(effects
+				(font
+					(size 1.27 1.27)
+				)
+				(hide yes)
+			)
+		)
+		(pin "1"
+		)
+		(pin "2"
+		)
+		(instances
+			(project ""
+				(path "/ce36a1c2-88cc-4cba-88a9-6235c3ec0ad6"
+					(reference "XTAL1")
+					(unit 1)
+				)
+			)
+		)
+	)
+	(symbol
 		(lib_id "adafruit:R-US_R0603")
 		(at 210.82 447.04 180)
@@
 			)
 		)
-		(property "Value" "27 pF"
+		(property "Value" "20 pF"
 			(at 805.18 415.2899 0)
 			(effects
@@
 					(unit 1)
 				)
-			)
-		)
-	)
-	(symbol
-		(lib_id "FC-135_32.7680KA-A0:FC-135_32.7680KA-A0")
-		(at 819.15 403.86 0)
-		(unit 1)
-		(exclude_from_sim no)
-		(in_bom yes)
-		(on_board yes)
-		(dnp no)
-		(fields_autoplaced yes)
-		(property "Reference" "Y2"
-			(at 819.15 393.7 0)
-			(effects
-				(font
-					(size 1.27 1.27)
-				)
-			)
-		)
-		(property "Value" "FC-135_32.7680KA-A0"
-			(at 819.15 396.24 0)
-			(effects
-				(font
-					(size 1.27 1.27)
-				)
-			)
-		)
-		(property "Footprint" "XTAL_FC-135_32.7680KA-A0"
-			(at 819.15 403.86 0)
-			(effects
-				(font
-					(size 1.27 1.27)
-				)
-				(justify left bottom)
-			)
-		)
-		(property "Datasheet" ""
-			(at 819.15 403.86 0)
-			(effects
-				(font
-					(size 1.27 1.27)
-				)
-				(justify left bottom)
-				(hide yes)
-			)
-		)
-		(property "Description" "32.7680 Khz 20ppm 12.5pf"
-			(at 819.15 403.86 0)
-			(effects
-				(font
-					(size 1.27 1.27)
-				)
-				(justify left bottom)
-				(hide yes)
-			)
-		)
-		(property "MF" "EPSON"
-			(at 819.15 403.86 0)
-			(effects
-				(font
-					(size 1.27 1.27)
-				)
-				(justify left bottom)
-				(hide yes)
-			)
-		)
-		(property "PACKAGE" "SMD-2 Epson"
-			(at 819.15 403.86 0)
-			(effects
-				(font
-					(size 1.27 1.27)
-				)
-				(justify left bottom)
-				(hide yes)
-			)
-		)
-		(property "PRICE" "0.33 USD"
-			(at 819.15 403.86 0)
-			(effects
-				(font
-					(size 1.27 1.27)
-				)
-				(justify left bottom)
-				(hide yes)
-			)
-		)
-		(property "Package" "SMD-2 Epson"
-			(at 819.15 403.86 0)
-			(effects
-				(font
-					(size 1.27 1.27)
-				)
-				(justify left bottom)
-				(hide yes)
-			)
-		)
-		(property "Check_prices" "https://www.snapeda.com/parts/FC-135%2032.7680KA-A0/EPSON/view-part/?ref=eda"
-			(at 819.15 403.86 0)
-			(effects
-				(font
-					(size 1.27 1.27)
-				)
-				(justify left bottom)
-				(hide yes)
-			)
-		)
-		(property "STANDARD" "Manufacturer Recommendation"
-			(at 819.15 403.86 0)
-			(effects
-				(font
-					(size 1.27 1.27)
-				)
-				(justify left bottom)
-				(hide yes)
-			)
-		)
-		(property "SnapEDA_Link" "https://www.snapeda.com/parts/FC-135%2032.7680KA-A0/EPSON/view-part/?ref=snap"
-			(at 819.15 403.86 0)
-			(effects
-				(font
-					(size 1.27 1.27)
-				)
-				(justify left bottom)
-				(hide yes)
-			)
-		)
-		(property "MP" "FC-135 32.7680KA-A0"
-			(at 819.15 403.86 0)
-			(effects
-				(font
-					(size 1.27 1.27)
-				)
-				(justify left bottom)
-				(hide yes)
-			)
-		)
-		(property "Price" "None"
-			(at 819.15 403.86 0)
-			(effects
-				(font
-					(size 1.27 1.27)
-				)
-				(justify left bottom)
-				(hide yes)
-			)
-		)
-		(property "Availability" "In Stock"
-			(at 819.15 403.86 0)
-			(effects
-				(font
-					(size 1.27 1.27)
-				)
-				(justify left bottom)
-				(hide yes)
-			)
-		)
-		(property "AVAILABILITY" "Good"
-			(at 819.15 403.86 0)
-			(effects
-				(font
-					(size 1.27 1.27)
-				)
-				(justify left bottom)
-				(hide yes)
-			)
-		)
-		(property "Description_1" "\\n                        \\n                            32.768 kHz ±20ppm Crystal 12.5pF 70 kOhms 2-SMD, No Lead\\n                        \\n"
-			(at 819.15 403.86 0)
-			(effects
-				(font
-					(size 1.27 1.27)
-				)
-				(justify left bottom)
-				(hide yes)
-			)
-		)
-		(pin "1"
-		)
-		(pin "2"
-		)
-		(instances
-			(project "Ember_v1.0"
-				(path "/ce36a1c2-88cc-4cba-88a9-6235c3ec0ad6"
-					(reference "Y2")
-					(unit 1)
-				)

Commit message: Added pilot board
Parts:
- added U5: ~, TESEO-LIV3F:TESEO-LIV3F, symbol TESEO-LIV3F:TESEO-LIV3F
Connections:
- new net: U5.10 (GND_RF), U5.12 (GND_RF)
Other:
- moved on the sheet: C1, C2, C3, C4, C5, C6, C7, C8, C9, IC1, L1, R1

Commit message: power supply changes to LDO
Parts:
- removed Buck_converter1: 4.7uH, SRN6045-4R7Y:SRN6045, symbol SRN6045-4R7Y:SRN6045-330M6045
- removed C20, C21, C23: 22uF, microbuilder:0603, symbol microbuilder:CAP_CERAMIC0603
- removed C22: 100nF, microbuilder:0603, symbol microbuilder:CAP_CERAMIC0603
- removed IC2: MP2315S, MP2315SGJ-Z:SOT65P280X100-8N, symbol MP2315SGJ-Z:MP2315SGJ-Z
- removed R10, R8: 100k, adafruit:R0603, symbol adafruit:R-US_R0603
- removed R11: 31.6k, adafruit:R0603, symbol adafruit:R-US_R0603
- removed R12: 20k, adafruit:R0603, symbol adafruit:R-US_R0603
- removed R6: 499k, adafruit:R0603, symbol adafruit:R-US_R0603
- removed R7: 10, adafruit:R0603, symbol adafruit:R-US_R0603
- removed R9: 9.09k, adafruit:R0603, symbol adafruit:R-US_R0603
- removed U5: ~, TESEO-LIV3F:TESEO-LIV3F, symbol TESEO-LIV3F:TESEO-LIV3F
- added U6: ~, AMS1117-3.3:SOT229P700X180-4N, symbol AMS1117-3.3:AMS1117-3.3
- C1, C10, C16, C2, C3, C4, C6: value 100nF -> 100 nF
- C13: value 10 uF -> 100 nF
- C17: value 3.3pF -> ~
- C18, C19: value 100nF -> ~
- C5: value 1uF -> 1 uF
- C7, C8, C9: value 4.7uF -> 4.7 uF
- L1: value 3.3uH -> 3.3 uH
- R15: value 10k -> 10 kohm
- R16: value 0 -> 0 ohm
- R19, R20, R21, R22, R23, R24: value 10k ohm -> 10 kohm
Connections:
- net BST is gone; now on net GND: C18.2 (P$2)
- net V_CC_AAM is gone; now on net GND: C19.2 (P$2)
- net 3v3: now also C17.1 (P$1), C18.1 (P$1), U6.2 (VOUT), U6.4 (VOUT); no longer C17.2 (P$2)
- net GND: now also C17.2 (P$2), U6.1 (ADJ/GND); no longer C19.1 (P$1), R13.2
- net V_MUX_OUT: now also C19.1 (P$1), U6.3 (VIN)
Other:
- moved on the sheet: C1, C10, C11, C12, C13, C14, C15, C16, C2, C24, C25, C3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

Commit message: Updated hirarchy and structure
Parts:
- removed C1, C10, C13, C16, C2, C3, C4, C6: 100 nF, microbuilder:0603, symbol microbuilder:CAP_CERAMIC0603
- removed C11, C12: 18pF, microbuilder:0603, symbol microbuilder:CAP_CERAMIC0603
- removed C14, C15: 10 uF, microbuilder:0603, symbol microbuilder:CAP_CERAMIC0603
- removed C17, C18, C19: ~, microbuilder:0603, symbol microbuilder:CAP_CERAMIC0603
- removed C24, C25: 20 pF, microbuilder:0603, symbol microbuilder:CAP_CERAMIC0603
- removed C5: 1 uF, microbuilder:0603, symbol microbuilder:CAP_CERAMIC0603
- removed C7, C8, C9: 4.7 uF, microbuilder:0603, symbol microbuilder:CAP_CERAMIC0603
- removed D1, D2: RSX501LAM20TR, RSX501LAM20TR:DIOM4725X105N, symbol RSX501LAM20TR:RSX501LAM20TR
- removed IC1: ~, RP2354B:QFN40P1000X1000X90-81N, symbol RP2354B:RP2354B
- removed J1: USB_C, USB4110GFA:GCT_USB4110GFA, symbol USB4110GFA:USB4110GFA
- removed J2: BATT_CONN, XT60-M:AMASS_XT60-M, symbol XT60-M:XT60-M
- removed L1: 3.3 uH, LQM2MPN3R3NG0L:LQM2MPN1R0NG0L, symbol LQM2MPN3R3NG0L:LQM2MPN3R3NG0L
- removed LED1: V_BATT, adafruit:CHIP-LED0603, symbol adafruit:LEDCHIP-LED0603
- removed LED2: VBUS, adafruit:CHIP-LED0603, symbol adafruit:LEDCHIP-LED0603
- removed R1: ~, adafruit:R0603, symbol adafruit:R-US_R0603
- removed R13, R14: 100, adafruit:R0603, symbol adafruit:R-US_R0603
- removed R15: 10 kohm, microbuilder:0603, symbol microbuilder:RESISTOR0603
- removed R16: 0 ohm, microbuilder:0603, symbol microbuilder:RESISTOR0603
- removed R17: ~, microbuilder:0603, symbol microbuilder:RESISTOR0603
- removed R18: 1k, microbuilder:0603, symbol microbuilder:RESISTOR0603
- removed R19, R20, R21, R22, R23, R24: 10 kohm, adafruit:R0603, symbol adafruit:R-US_R0603
- removed R2, R3: 5.1k, adafruit:R0603, symbol adafruit:R-US_R0603
- removed R4, R5: 27.4, adafruit:R0603, symbol adafruit:R-US_R0603
- removed S1: ~, DTS-3:DTS-3, symbol DTS-3:DTS-3
- removed U1: FLASH_128K, W25Q32JVSSIQ:SOIC127P790X216-8N, symbol W25Q32JVSSIQ:W25Q32JVSSIQ
- removed U2: BNO055, Package_LGA:LGA-28_5.2x3.8mm_P0.5mm, symbol Sensor_Motion:BNO055
- removed U3: ~, kx134:LGA12_2X2X0P9_ROM, symbol kx134:KX134-1211
- removed U4: BMP280, Package_LGA:Bosch_LGA-8_2x2.5mm_P0.65mm_ClockwisePinNumbering, symbol Sensor_Pressure:BMP280
- removed U6: ~, AMS1117-3.3:SOT229P700X180-4N, symbol AMS1117-3.3:AMS1117-3.3
- removed XTAL1: XTAL_FC135, Q13FC1350000400:XTAL_FC-135_EPS, symbol Q13FC1350000400:Q13FC1350000400
- removed Y1: ~, YSX321SL:YSX321SL, symbol YSX321SL:YSX321SL
Other:
- added sheet Main_board (main.kicad_sch)
- added sheet RF_board (rf_board.kicad_sch)
- note removed: "BMP"
- note removed: "BNO"
- note removed: "Crystal Oscillator"
- note removed: "External Flash"
- note removed: "FLASH"
- note removed: "Internal Flash Bootsel"
- note removed: "KX"
- note removed: "PULL UPS"
- note removed: "Power Supply"
