File: Ember_v1.0/Ember_v1.0.kicad_pcb (KiCad board)
At the start: 2 copper layers, 66 parts, among them IC2 MP2315S, J1 USB_C, J2 BATT_CONN, U1 FLASH_128K, U2 BNO055, U4 BMP280

Commit message: Base requirements added in schemcatics
Parts:
- removed Buck_converter1: 4.7uH, SRN6045-4R7Y:SRN6045
- removed IC2: MP2315S, MP2315SGJ-Z:SOT65P280X100-8N
- removed R10: 100k, adafruit:R0603
- removed R11: 31.6k, adafruit:R0603
- removed R12: 20k, adafruit:R0603
- removed R9: 9.09k, adafruit:R0603
- added C26: ~, microbuilder:0603, F.Cu at (44.9, 36.1)
- added C27: ~, microbuilder:0603, F.Cu at (44.9, 38.7)
- added C28: ~, microbuilder:0603, F.Cu at (44.9, 41.3)
- added FL1: Saw_filter, AFS14A04-1575.42-T3:FIL_AFS14A04-1575.42-T3, F.Cu at (50.7, 62.3)
- added J3: DROGUE, OSTTA020161:ONSHORE_OSTTA020161, F.Cu at (29.3, 41.5)
- added J4: ~, sma-connector:RFSOLUTIONS_CON-SMA-EDGE-S, F.Cu at (83.5, 39.0)
- added J5: MAIN, OSTTA020161:ONSHORE_OSTTA020161, F.Cu at (29.3, 53.0)
- added J6: MAN2, OSTTA020161:ONSHORE_OSTTA020161, F.Cu at (29.3, 64.4)
- added J7: DROGUE2, OSTTA020161:ONSHORE_OSTTA020161, F.Cu at (29.3, 75.9)
- added J8: ARM, OSTTA020161:ONSHORE_OSTTA020161, F.Cu at (29.3, 87.3)
- added J9: ~, sma-connector:RFSOLUTIONS_CON-SMA-EDGE-S, F.Cu at (83.5, 47.4)
- added L2: ~, microbuilder:0603, F.Cu at (51.3, 59.6)
- added Q1: SISA96DN-T1, SISA96DN-T1-GE3:SIS862DNT1GE3, F.Cu at (39.3, 37.8)
- added Q2: SISA96DN-T1, SISA96DN-T1-GE3:SIS862DNT1GE3, F.Cu at (39.3, 44.0)
- added Q3: SISA96DN-T1, SISA96DN-T1-GE3:SIS862DNT1GE3, F.Cu at (39.3, 50.1)
- added Q4: SISA96DN-T1, SISA96DN-T1-GE3:SIS862DNT1GE3, F.Cu at (39.3, 56.3)
- added R28: 33k, microbuilder:0603, F.Cu at (44.9, 43.9)
- added R29: 1k, microbuilder:0603, F.Cu at (44.9, 46.5)
- added R30: 33k, microbuilder:0603, F.Cu at (44.9, 49.1)
- added R31: 1k, microbuilder:0603, F.Cu at (44.9, 51.7)
- added R32: 33k, microbuilder:0603, F.Cu at (44.9, 54.3)
- added R33: 1k, microbuilder:0603, F.Cu at (44.9, 56.9)
- added U5: Teseo_liv3f, TESEO-LIV3F:TESEO-LIV3F, F.Cu at (77.2, 58.5)
- added U6: ~, AMS1117-3.3:SOT229P700X180-4N, F.Cu at (39.9, 64.1)
- added U7: Waveshare_SX1262, CORE1262-868M:XCVR_CORE1262-868M, F.Cu at (60.6, 46.5)
- added U8: ~, AMS1117-5.0:SOT229P700X180-4N, F.Cu at (40.4, 74.0)
- C1, C10, C16, C2, C3, C4, C6: value 100nF -> 100 nF
- C13: value 10 uF -> 100 nF
- C17: value 3.3pF -> ~
- C18, C19: value 100nF -> ~
- C20, C23: value 22uF -> 120 pF
- C21: value 22uF -> 10 uF
- C22: value 100nF -> 120 pF
- C5: value 1uF -> 1 uF
- C7, C8, C9: value 4.7uF -> 4.7 uF
- L1: value 3.3uH -> 3.3 uH
- R15: value 10k -> 10 kohm
- R16: value 0 -> 0 ohm
- R19, R20, R21, R22, R23, R24: value 10k ohm -> 10 kohm
- R6: value 499k -> 33k; footprint adafruit:R0603 -> microbuilder:0603
- R7: value 10 -> 1k; footprint adafruit:R0603 -> microbuilder:0603
- R8: value 100k -> 4.7k; footprint adafruit:R0603 -> microbuilder:0603
- moved R3 124.0 mm to (174.2, 41.6), turned to 180 degrees
- moved R5 123.6 mm to (169.7, 41.9), turned to 90 degrees
- moved R4 120.2 mm to (167.6, 41.9), turned to 90 degrees
- moved C8 119.3 mm to (184.6, 66.8)
- moved S1 117.8 mm to (157.7, 36.1), turned to 90 degrees
- moved R2 113.7 mm to (163.7, 41.4), turned to 180 degrees
- moved R1 112.9 mm to (179.8, 77.8)
- moved C7 112.0 mm to (179.6, 74.4)
- moved C1 112.0 mm to (178.5, 54.4)
- moved C2 110.8 mm to (177.4, 57.0)
- moved C3 110.5 mm to (177.0, 59.5)
- moved C6 110.3 mm to (176.8, 67.5)
- moved C4 110.3 mm to (176.9, 62.9)
- moved C5 110.1 mm to (176.8, 65.7)
- moved C9 105.3 mm to (179.1, 70.7)
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Connections:
- net /1v1 renamed /Main_board/1v1
- net /D_M renamed /Main_board/D_N
- net /D_P renamed /Main_board/D_P
- net /FLASH_EXT_CS renamed /Main_board/FLASH_EXT_CS
- net /QSPI_SCLK renamed /Main_board/QSPI_SCLK
- net /QSPI_SD0 renamed /Main_board/QSPI_SD0
- net /QSPI_SD1 renamed /Main_board/QSPI_SD1
- net /QSPI_SD2 renamed /Main_board/QSPI_SD2
- net /QSPI_SD3 renamed /Main_board/QSPI_SD3
- net /QSPI_SS renamed /Main_board/QSPI_SS
- net /SCL renamed /Main_board/SCL
- net /SDA renamed /Main_board/SDA
- net /VBUS renamed /Main_board/VBUS
- net /XIN renamed /Main_board/XIN
- net /XIN32 renamed /Main_board/XIN32
- net /XOUT renamed /Main_board/XOUT
- net /XOUT32 renamed /Main_board/XOUT32
- C1 pad 1: /3v3 -> /Main_board/3v3
- C1 pad 2: /GND -> /Main_board/GND
- C10 pad 1: /3v3 -> /Main_board/3v3
- C10 pad 2: /GND -> /Main_board/GND
- C11 pad 2: /GND -> /Main_board/GND
- C12 pad 1: /GND -> /Main_board/GND
- C13 pad 1: /GND -> /Main_board/GND
- C13 pad 2: /3v3 -> /Main_board/3v3
- C14 pad 1: /3v3 -> /Main_board/3v3
- C14 pad 2: /GND -> /Main_board/GND
- C15 pad 1: /3v3 -> /Main_board/3v3
- C15 pad 2: /GND -> /Main_board/GND
- C16 pad 1: /GND -> /Main_board/GND
- C17 pad 1: Net-(C17-P$1) -> /Main_board/3v3
- C17 pad 2: /3v3 -> /Main_board/GND
- C18 pad 1: Net-(C18-P$1) -> /Main_board/3v3
- C18 pad 2: /BST -> /Main_board/GND
- C19 pad 1: /GND -> /Main_board/V_MUX_OUT
- C19 pad 2: /V_CC_AAM -> /Main_board/GND
- C2 pad 1: /3v3 -> /Main_board/3v3
- C2 pad 2: /GND -> /Main_board/GND
- C20 pad 1: /GND -> /RF_board/SAW_OUT
- C20 pad 2: /3v3 -> /RF_board/GPS_RF_IN
- C21 pad 1: /GND -> /RF_board/GND
- C21 pad 2: /3v3 -> /RF_board/3v3
- C22 pad 1: /GND -> /RF_board/GPS_ANT
- C22 pad 2: /V_MUX_OUT -> /RF_board/SAW_IN
- C23 pad 1: /GND -> /RF_board/GND
- C23 pad 2: /V_MUX_OUT -> /RF_board/GPS_ANT
- C24 pad 1: /GND -> /Main_board/GND
- C25 pad 1: /GND -> /Main_board/GND
- C3 pad 1: /3v3 -> /Main_board/3v3
- C3 pad 2: /GND -> /Main_board/GND
- C4 pad 1: /3v3 -> /Main_board/3v3
- C4 pad 2: /GND -> /Main_board/GND
- C5 pad 2: /GND -> /Main_board/GND
- C6 pad 2: /GND -> /Main_board/GND
- C7 pad 2: /GND -> /Main_board/GND
- C8 pad 2: /GND -> /Main_board/GND
- C9 pad 1: /3v3 -> /Main_board/3v3
- C9 pad 2: /GND -> /Main_board/GND
- D1 pad 1: /V_MUX_OUT -> /Main_board/V_MUX_OUT
- D1 pad 2: /V_BATT -> /Main_board/5v
- D2 pad 1: /V_MUX_OUT -> /Main_board/V_MUX_OUT
- IC1 pad 15: /3v3 -> /Main_board/3v3
- IC1 pad 24: /3v3 -> /Main_board/3v3
- IC1 pad 29: /3v3 -> /Main_board/3v3
- IC1 pad 35: /3v3 -> /Main_board/3v3
- IC1 pad 41: /3v3 -> /Main_board/3v3
- IC1 pad 5: /3v3 -> /Main_board/3v3
- IC1 pad 50: /3v3 -> /Main_board/3v3
- IC1 pad 59: /3v3 -> /Main_board/3v3
- IC1 pad 60: /3v3 -> /Main_board/3v3
- IC1 pad 62: /GND -> /Main_board/GND
- IC1 pad 64: /3v3 -> /Main_board/3v3
- IC1 pad 68: /3v3 -> /Main_board/3v3
- IC1 pad 69: /3v3 -> /Main_board/3v3
- IC1 pad 76: /3v3 -> /Main_board/3v3
- IC1 pad 81: /GND -> /Main_board/GND
- J1 pad A1/B12: /GND -> /Main_board/GND
- J1 pad A6: Net-(J1-DP1) -> /Main_board/D_Pr
- J1 pad A7: Net-(J1-DN1) -> /Main_board/D_Nr
- J1 pad B1/A12: /GND -> /Main_board/GND
- J1 pad B6: unconnected-(J1-DP2-PadB6) -> /Main_board/D_Pr
- J1 pad B7: unconnected-(J1-DN2-PadB7) -> /Main_board/D_Nr
- J1 pad S1: /GND -> /Main_board/GND
- J1 pad S2: /GND -> /Main_board/GND
- J1 pad S3: /GND -> /Main_board/GND
- J1 pad S4: /GND -> /Main_board/GND
- J2 pad N: /GND -> /Main_board/GND
- J2 pad P: /V_BATT -> /Main_board/V_BATT
- LED1 pad A: /V_BATT -> /Main_board/5v
- R1 pad 2: /3v3 -> /Main_board/3v3
- R13 pad 2: /GND -> unconnected-(R13-Pad2)
- R14 pad 2: /GND -> /Main_board/GND
- R15 pad 2: /3v3 -> /Main_board/3v3
- R19 pad 1: /GND -> /Main_board/GND
- R2 pad 2: /GND -> /Main_board/GND
- R20 pad 1: /3v3 -> /Main_board/3v3
- R21 pad 1: /3v3 -> /Main_board/3v3
- R22 pad 1: /3v3 -> /Main_board/3v3
- R23 pad 1: /GND -> /Main_board/GND
- R24 pad 1: /3v3 -> /Main_board/3v3
- R3 pad 1: /GND -> /Main_board/GND
- R4 pad 2: Net-(J1-DP1) -> /Main_board/D_Pr
- R5 pad 2: Net-(J1-DN1) -> /Main_board/D_Nr
- R6 pad 1: Net-(IC2-EN) -> Net-(Q4-G)
- R6 pad 2: /V_MUX_OUT -> /Main_board/GND
- R7 pad 1: Net-(IC2-BST) -> /Main_board/DROGUE2
- R7 pad 2: Net-(C18-P$1) -> Net-(Q4-G)
- R8 pad 1: Net-(IC2-AAM) -> /RF_board/GND
- R8 pad 2: /V_CC_AAM -> /RF_board/LORA_CS
- S1 pad 2: /GND -> /Main_board/GND
- U1 pad 4: /GND -> /Main_board/GND
- U1 pad 8: /3v3 -> /Main_board/3v3
- U2 pad 18: /GND -> /Main_board/GND
- U2 pad 2: /GND -> /Main_board/GND
- U2 pad 25: /GND -> /Main_board/GND
- U2 pad 28: /3v3 -> /Main_board/3v3
- U2 pad 3: /3v3 -> /Main_board/3v3
- U2 pad 4: /3v3 -> /Main_board/3v3
- U2 pad 5: /GND -> /Main_board/GND
- U2 pad 6: /GND -> /Main_board/GND
- U3 pad 1: /3v3 -> /Main_board/3v3
- U3 pad 10: /3v3 -> /Main_board/3v3
- U3 pad 3: /3v3 -> /Main_board/3v3
- U3 pad 4: /GND -> /Main_board/GND
- U3 pad 7: /3v3 -> /Main_board/3v3
- U3 pad 8: /GND -> /Main_board/GND
- U3 pad 9: /GND -> /Main_board/GND
- U4 pad 1: /GND -> /Main_board/GND
- U4 pad 6: /3v3 -> /Main_board/3v3
- U4 pad 7: /GND -> /Main_board/GND
- U4 pad 8: /3v3 -> /Main_board/3v3
- Y1 pad 2: /GND -> /Main_board/GND
- Y1 pad 4: /GND -> /Main_board/GND
Routing:
- net /Main_board/QSPI_SD3: track 0.00 -> 22.2 mm
- net /Main_board/QSPI_SCLK: track 0.00 -> 20.0 mm
- net /Main_board/D_P: track 0.00 -> 19.2 mm
- net /Main_board/D_N: track 0.00 -> 19.2 mm
- net /Main_board/QSPI_SD1: track 0.00 -> 18.3 mm
- net /Main_board/QSPI_SD2: track 0.00 -> 16.7 mm
- net /Main_board/QSPI_SD0: track 0.00 -> 16.7 mm
- net /Main_board/3v3: track 0.00 -> 7.12 mm
- net /Main_board/D_Nr: track 0.00 -> 5.70 mm
- net /Main_board/D_Pr: track 0.00 -> 5.54 mm
- net Net-(U1-~{CS}): track 0.00 -> 5.23 mm
Other:
- copper layers 2 -> 4

Commit message: Added everything till test launch 1 prep
Parts:
- moved J2 48.8 mm to (143.0, 117.5)
Changed lines of the file:
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@@
 	(footprint "XT60-M:AMASS_XT60-M"
 		(layer "F.Cu")
-		(at 95.3235 107.155)
+		(at 143.02 117.48)
 		(property "Reference" "J2"
 			(at -8 -5.3 0)
