File: Ember_v1.0/main.kicad_sch (KiCad schematic)
At the start: 75 parts, among them J1 USB_C, J2 BATT_CONN, J3 DROGUE, J5 MAIN, J6 MAN2, J7 DROGUE2, J8 ARM, Q1 SISA96DN-T1, Q2 SISA96DN-T1, Q3 SISA96DN-T1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

Commit message: Base requirements added in schemcatics
Connections:
- net D_Nr: now reaches J1.A7 (DN1), R5.2
- net D_Nr: now also J1.B7 (DN2)
- net D_Pr: now reaches J1.A6 (DP1), R4.2
- net D_Pr: now also J1.B6 (DP2)
- net D_M renamed D_N
Changed lines of the file:
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@@
+	(wire
+		(pts
+			(xy 63.5 72.39) (xy 63.5 74.93)
+		)
+		(stroke
+			(width 0)
+			(type default)
+		)
+	)
 	(wire
 		(pts
@@
 	(wire
 		(pts
+			(xy 60.96 72.39) (xy 60.96 74.93)
+		)
+		(stroke
+			(width 0)
+			(type default)
+		)
+	)
+	(wire
+		(pts
 			(xy 220.98 365.76) (xy 223.52 365.76)
 		)
@@
 		)
 	)
-	(label "D_M"
+	(label "D_N"
 		(at 355.6 182.88 0)
 		(effects
@@
 		)
 	)
+	(label "D_Pr"
+		(at 60.96 72.39 180)
+		(effects
+			(font
+				(size 1.27 1.27)
+			)
+			(justify right bottom)
+		)
+	)
 	(label "GND"
 		(at 52.07 330.2 180)
@@
 		)
 	)
-	(label "D_M"
+	(label "D_N"
 		(at 71.12 130.81 0)
 		(effects
@@
 		)
 	)
+	(label "D_Nr"
+		(at 63.5 72.39 0)
+		(effects
+			(font
+				(size 1.27 1.27)
+			)
+			(justify left bottom)
+		)
+	)
 	(label "GND"
 		(at 142.24 191.77 0)
@@
 		)
 	)
+	(label "D_Pr"
+		(at 60.96 115.57 0)
+		(effects
+			(font
+				(size 1.27 1.27)
+			)
+			(justify left bottom)
+		)
+	)
 	(label "QSPI_SD1"
 		(at 335.28 181.61 90)
@@
 		)
 	)
+	(label "D_Nr"
+		(at 71.12 114.3 0)
+		(effects
+			(font
+				(size 1.27 1.27)
+			)
+			(justify left bottom)
+		)
+	)

Commit message: Added everything till test launch 1 prep
Parts:
- removed R19, R20, R21, R22, R23, R24: 10 kohm, adafruit:R0603, symbol adafruit:R-US_R0603
- added C30: ~, microbuilder:0603, symbol microbuilder:CAP_CERAMIC0603
- added R10, R11, R12, R19, R20, R24, R25, R9: 10k, microbuilder:0603, symbol microbuilder:RESISTOR0603
- added U9: BMI160, Package_LGA:Bosch_LGA-14_3x2.5mm_P0.5mm, symbol Sensor_Motion:BMI160
- C13: value 100 nF -> 100n
- C14: value 10 uF -> 100n
Connections:
- net 3v3: now also C30.1 (P$1), R10.1, R12.1, R20.1, R24.1, R25.1, R9.2, U9.5 (VDDIO), U9.8 (VDD); no longer U3.1 (SDO/ADDR)
- net GND: now also C30.2 (P$2), R11.1, R19.2
- net SCL: now also R24.2
- net SDA: now also R12.2
- net at U4.2 (CSB): now also R10.2
- net at U4.5 (SDO): now also R11.2
- net at U2.11 (~{RESET}): now also R25.2
- net BNO_INT: now reaches U2.14 (INT)
- net at U2.17 (COM3): now also R19.1
- new net: R20.2, U3.1 (SDO/ADDR)
- new net: R9.1, U9.1 (SDO)
