File: Ember_RF_v0/Ember_RF_v0.kicad_sch (KiCad schematic)
At the start: 26 parts, among them Q2 SISA96DN-T1, Q5 CJ3400

Commit message: v0.2 and RF v0 sent for fab - Lisan Al-gaib
Parts:
- added C6, C7: 100nF, microbuilder:0603, symbol microbuilder:CAP_CERAMIC0603
- added D1: RSX501LAM20TR, RSX501LAM20TR:DIOM4725X105N, symbol RSX501LAM20TR:RSX501LAM20TR
- C5: value 100nF -> 10uF
Connections:
- net 3v3: now also C6.1 (P$1)
- net 5v: now also C7.2 (P$2)
- net GND: now also C6.2 (P$2), C7.1 (P$1)
- net V_BATT: now also D1.2; no longer C4.1 (P$1), IC1.2 (EN), IC1.3 (VIN)
- new net: C4.1 (P$1), D1.1, IC1.2 (EN), IC1.3 (VIN)
Other:
- moved on the sheet: C4, LED1, R17
