File: Ember_v0.2/Ember_v0.2.kicad_pcb (KiCad board)
At the start: 2 copper layers, 75 x 99.5 mm, 114 parts, among them J3 DROGUE, J4 BATT_CONN, J5 MAIN, J6 MAN2, J7 DROGUE2, J8 ARM, Q1 SISA96DN-T1, Q2 SISA96DN-T1, Q3 SISA96DN-T1, Q4 SISA96DN-T1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

Commit message: All changes and things are done in both FCU and TDU - Lisan Al-gaib!
Parts:
- removed the ? at (81.0, 106.0)
- removed the ? at (81.0, 131.0)
- removed the ? at (81.0, 92.0)
- removed the ? at (81.0, 117.0)
- removed JP6: ~, microbuilder:1X02_OVAL
- removed Q6: SISA96DN-T1, SISA96DN-T1-GE3:SIS862DNT1GE3
- removed R23: 33k, microbuilder:0603
- removed R24: 1k, microbuilder:0603
- removed the REF** at (150.0, 99.8)
- removed the REF** at (85.6, 53.0)
- removed the REF** at (147.6, 139.5)
- removed the REF** at (149.9, 119.7)
- removed the REF** at (85.6, 139.5)
- removed the REF** at (111.9, 99.7)
- removed the REF** at (147.6, 53.0)
- added ?: , drogue_label:DROGUE0, F.Cu at (81.2, 105.8)
- added ?: , main_label:MAIN0, F.Cu at (81.2, 92.3)
- added ?: , main_label:MAIN0, F.Cu at (81.2, 117.0)
- added ?: , drogue_label:DROGUE0, F.Cu at (81.2, 130.5)
- added G***: LOGO, RT_Graphics:strain_gauge_label, F.Cu at (111.9, 141.4)
- added G***: LOGO, RT_Graphics:iitb_logo, F.Cu at (148.0, 71.5)
- added REF**: MountingHole_3.2mm_M3_DIN965_Pad, MountingHole:MountingHole_3.2mm_M3_DIN965_Pad, F.Cu at (147.6, 53.0)
- added REF**: MountingHole_3.2mm_M3_DIN965_Pad, MountingHole:MountingHole_3.2mm_M3_DIN965_Pad, F.Cu at (111.9, 99.7)
- added REF**: MountingHole_3.2mm_M3_DIN965_Pad, MountingHole:MountingHole_3.2mm_M3_DIN965_Pad, F.Cu at (147.6, 139.5)
- added REF**: MountingHole_3.2mm_M3_DIN965_Pad, MountingHole:MountingHole_3.2mm_M3_DIN965_Pad, F.Cu at (149.9, 119.7)
- added REF**: MountingHole_3.2mm_M3_DIN965_Pad, MountingHole:MountingHole_3.2mm_M3_DIN965_Pad, F.Cu at (85.6, 53.0)
- added REF**: MountingHole_3.2mm_M3_DIN965_Pad, MountingHole:MountingHole_3.2mm_M3_DIN965_Pad, F.Cu at (149.9, 99.7)
- added REF**: MountingHole_3.2mm_M3_DIN965_Pad, MountingHole:MountingHole_3.2mm_M3_DIN965_Pad, F.Cu at (85.6, 139.5)
- moved REF** 64.8 mm to (95.6, 52.4), turned to 0 degrees
- moved G*** 20.5 mm to (137.3, 71.7)
- moved G*** 20.0 mm to (114.8, 63.6)
- moved ? 0.41 mm to (136.6, 57.8)
- moved ? 0.33 mm to (134.0, 57.6)
- moved ? 0.33 mm to (128.9, 58.5)
- moved ? 0.30 mm to (131.5, 58.8)
Connections:
- U7 pad P$5: /CAM -> unconnected-(U7-GP3-PadP$5)
Routing:
- net /V_BATT: track 153.6 -> 73.0 mm
- net /CAM: track 58.4 -> 0.00 mm
- net /CAM_OUT: track 6.57 -> 0.00 mm
- net Net-(Q6-G): track 5.77 -> 0.00 mm
- net /GND: track 34.9 -> 30.5 mm, vias 46 -> 47
- net /ACT1: track 23.4 -> 22.2 mm

Commit message: v0.2 and RF v0 sent for fab - Lisan Al-gaib
Parts:
- added G***: LOGO, RT_Graphics:solder_things, B.Cu at (146.1, 109.7)
- added G***: LOGO, RT_Graphics:daft_punk, B.Cu at (144.8, 119.6)
- moved G*** 0.35 mm to (127.4, 93.8)
Connections:
- REF** pad 1: (no net) -> /GND (x7)
Routing:
- net /DROGUE: track 47.9 -> 48.5 mm
Other:
- board text added: "Can't stop Daft Punking at the lab"
- board text added: "I kept hating DRC errors until it was a significant one T~T - The same guy who hates uPy's type handling and refers DRC errors as KiCad tantrums"
- board text added: "It'll start working as soon as my cortisol goes low - Someone who hates uPython's type handling"
- board text added: "It's gonna go up... And it's gonna come down too... - Some wise person"
- board text added: "The rocket knows where it is (probably) - Someone who says {dblquote}Tujhe prompt engineering nahi aata{dblquote}"
