File: Ember_ECU_V0/_restore_backup_2026-08-13T19-42-49-402/lre_avio_daq2.kicad_sch (KiCad schematic)
At the start: 124 parts, among them J1 Screw_Terminal_01x02, J10 Conn_01x03_Socket, J11 USB_C_Receptacle_USB2.0_16P, J12 XT30PW-F, J13 XT30PW-F, J14 XT30PW-F, J15 XT30PW-F, J16 XT30PW-F, J2 Conn_01x04, J3 XT60PW-M, J4 DB25_Socket, J5 Conn_01x03_Socket, J6 Conn_01x03_Socket, J7 Conn_01x03_Socket, J8 Conn_01x03_Socket, J9 Conn_01x03_Socket, Q2 SISA96DN-T1, Q3 SISA96DN-T1, Q4 SISA96DN-T1, SW1 SW_SPDT, U1 AMS1117-5.0, U10 ADS8353QPWRQ1, U11 ADS8353QPWRQ1, U12 STM32F412VGTx, U2 HX711, U3 SN65HVD230, U5 AMS1117-5.0, U6 ADS8353QPWRQ1, U7 MAX31856, U8 MAX31856, U9 MAX31856, Y1 8 MHz

Commit message: commit
Parts:
- removed J15, J16: XT30PW-F, xt30:CONN_XT30PW-F_AMA, symbol 2026-08-03_13-16-17:XT30PW-F
- removed Q3, Q4: SISA96DN-T1, SISA96DN-T1-GE3:SIS862DNT1GE3, symbol SISA96DN-T1-GE3:SISA96DN-T1-GE3
- removed R30, R32: 33k, Resistor_SMD:R_0201_0603Metric, symbol microbuilder:RESISTOR0603
- removed R31, R33: 1k, Resistor_SMD:R_0201_0603Metric, symbol microbuilder:RESISTOR0603
- J12, J13, J14: footprint xt30:CONN_XT30PW-F_AMA -> CONN_XT30PW-F_AMA
- R1, R10, R11, R12, R13, R14, R15, R16, R17, R18, R19, R2, R20, R21, R3, R4, R6, R7, R8, R9, SW1: footprint Resistor_SMD:R_0201_0603Metric -> (none)
- R28, R29: footprint Resistor_SMD:R_0201_0603Metric -> microbuilder:0603
- R5: footprint Resistor_SMD:R_0201_0603Metric -> RSX501LAM20TR:DIO_RB050LAM_ROM-L
Connections:
- net Conn: now reaches U12.17 (PC2)
- net Conn: now also R29.1
- net Conn1: no longer names the net of U12.81 (PD0)
- net Conn1: no longer R29.1
- net Conn2: no longer names the net of U12.82 (PD1)
- net Conn3: no longer names the net of U12.83 (PD2)
Other:
- moved on the sheet: C10, C11, C12, C13, J12, J13, J14, J2, Q2, R18, R19, R20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
