File: Ember_ECU_V0/lre_avio_daq2.kicad_sch (KiCad schematic)
At the start: 124 parts, among them J1 Screw_Terminal_01x02, J10 Conn_01x03_Socket, J11 USB_C_Receptacle_USB2.0_16P, J12 XT30PW-F, J13 XT30PW-F, J14 XT30PW-F, J15 XT30PW-F, J16 XT30PW-F, J2 Conn_01x04, J3 XT60PW-M, J4 DB25_Socket, J5 Conn_01x03_Socket, J6 Conn_01x03_Socket, J7 Conn_01x03_Socket, J8 Conn_01x03_Socket, J9 Conn_01x03_Socket, Q2 SISA96DN-T1, Q3 SISA96DN-T1, Q4 SISA96DN-T1, SW1 SW_SPDT, U1 AMS1117-5.0, U10 ADS8353QPWRQ1, U11 ADS8353QPWRQ1, U12 STM32F412VGTx, U2 HX711, U3 SN65HVD230, U5 AMS1117-5.0, U6 ADS8353QPWRQ1, U7 MAX31856, U8 MAX31856, U9 MAX31856, Y1 8 MHz

Commit message: erc issues and pcb related things resolved, still some remaining
Parts:
- C53, C54, C55, C56, C57, C58, C59, C60, C61, C62, C63: footprint (none) -> Capacitor_SMD:C_0201_0603Metric
Connections:
- net TC1_CS is gone; now on net SPI1_CS1: U12.29 (PA4)
- net TC2_CS is gone; now on net SPI1_CS2: U12.35 (PB0)
- net TC3_CS is gone; now on net SPI1_CS3: U12.36 (PB1)
- no-connect marks 12 -> 58
Other:
- moved on the sheet: C10, C11, C12, C13, J12, J13, J14, J15, J16, J2, J4, Q2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

Commit message: commit
Parts:
- C1, C10, C11, C12, C13, C14, C15, C16, C17, C18, C19, C2, C20, C21, C22, C23, C24, C25, C26, C27, C28, C3, C30, C35, C39, C4, C45, C46, C47, C48, C49, C5, C50, C51, C52, C6, C8, C9: footprint (none) -> Capacitor_SMD:C_0201_0603Metric
- D1, D2: footprint (none) -> footprints:SOD123FA_ONS
- J10, J5, J6, J7, J8, J9: footprint (none) -> Connector_Phoenix_GMSTB:PhoenixContact_GMSTBVA_2,5_3-G-7,62_1x03_P7.62mm_Vertical
Connections:
- net SPI1_CS1: no longer U12.29 (PA4)
- net SPI1_CS2: no longer U12.35 (PB0)
- net SPI1_CS3: no longer U12.36 (PB1)
- new net TC1_CS: U12.29 (PA4)
- new net TC2_CS: U12.35 (PB0)
- new net TC3_CS: U12.36 (PB1)
- no-connect marks 58 -> 12
Other:
- moved on the sheet: C10, C11, C12, C13, J12, J13, J14, J15, J16, J2, J4, Q2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

Commit message: ECU schematics updated
Parts:
- removed J1: Screw_Terminal_01x02, symbol Connector:Screw_Terminal_01x02
- removed J10, J5, J6, J7, J8, J9: Conn_01x03_Socket, Connector_Phoenix_GMSTB:PhoenixContact_GMSTBVA_2,5_3-G-7,62_1x03_P7.62mm_Vertical, symbol Connector:Conn_01x03_Socket
- removed J2: Conn_01x04, symbol Connector_Generic:Conn_01x04
- removed J4: DB25_Socket, symbol Connector:DB25_Socket
- removed Q4: SISA96DN-T1, SISA96DN-T1-GE3:SIS862DNT1GE3, symbol SISA96DN-T1-GE3:SISA96DN-T1-GE3
- removed TC1, TC2, TC3: Thermocouple, symbol Device:Thermocouple
- removed Y1: 8 MHz, symbol Device:Crystal
- added C31, C42, C64, C65, C68, C69: 10 muF, Capacitor_SMD:C_0201_0603Metric, symbol Device:C
- added C43, C44, C66, C67, C70, C71: 0.1 muF, Capacitor_SMD:C_0201_0603Metric, symbol Device:C
- added C72: 100 nF, Capacitor_SMD:C_0201_0603Metric, symbol Device:C
- added J1: Conn_01x02_Socket, Connector_JST:JST_EH_B2B-EH-A_1x02_P2.50mm_Vertical, symbol Connector:Conn_01x02_Socket
- added J17: SMPW-CC-K-M, SMPW-CC-K-M:SMPWCCKM, symbol SMPW-CC-K-M:SMPW-CC-K-M
- added J18, J19: SMPW-CC-K-M, SMPWCCKM, symbol SMPW-CC-K-M:SMPW-CC-K-M
- added J2, J24: DB25_Socket_MountingHoles, Connector_Dsub:DSUB-25_Socket_Horizontal_P2.77x2.84mm_EdgePinOffset4.94mm_Housed_MountingHolesOffset4.94mm, symbol Connector:DB25_Socket_MountingHoles
- added J23: DA15_Socket_MountingHoles, Connector_Dsub:DSUB-15_Socket_Horizontal_P2.77x2.84mm_EdgePinOffset4.94mm_Housed_MountingHolesOffset4.94mm, symbol Connector:DA15_Socket_MountingHoles
- added Q1: SISA96DN-T1-GE3, SIS862DNT1GE3, symbol SISA96DN-T1-GE3:SISA96DN-T1-GE3
- added R22, R23, R24, R25, R26, R27: 100, Resistor_SMD:R_0201_0603Metric, symbol Device:R
- added U13, U14, U4: HX711, Package_SO:SOIC-16_3.9x9.9mm_P1.27mm, symbol Analog_ADC:HX711
- added Y1: Crystal_8Mhz, Crystal:Crystal_SMD_7050-4Pin_7.0x5.0mm, symbol Device:Crystal_GND24
- D1, D2: footprint footprints:SOD123FA_ONS -> RSX501LAM20TR:DIO_RB050LAM_ROM
- Q2, Q3: value SISA96DN-T1 -> SISA96DN-T1-GE3; footprint SISA96DN-T1-GE3:SIS862DNT1GE3 -> SIS862DNT1GE3; Arrow Part Number (none) -> SISA96DN-T1-GE3; Arrow Price/Stock (none) -> https://www.arrow.com/en/products/sisa96dn-t1-ge3/vishay.ht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; Height (none) -> 1.12; Manufacturer_Name (none) -> Vishay; Manufacturer_Part_Number (none) -> SISA96DN-T1-GE3; Mouser Part Number (none) -> 78-SISA96DN-T1-GE3; Mouser Price/Stock (none) -> https://www.mouser.co.uk/ProductDetail/Vishay-Siliconix/SIS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
- SW1: footprint Resistor_SMD:R_0201_0603Metric -> Button_Switch_SMD:SW_SPDT_PCM12
Connections:
- net +3.3V is gone; now on net 3v3: C27.2, C28.2, R15.1, R16.1, U9.5 (AVDD), U9.8 (DVDD)
- net 3v3: now also U12.22 (VDDA), C31.2, C64.2, C68.2, C72.2, U13.1 (VSUP), U13.15 (RATE), U13.16 (DVDD), U13.2 (BASE), U14.1 (VSUP), U14.15 (RATE), U14.16 (DVDD), U14.2 (BASE), U4.1 (VSUP), U4.15 (RATE), U4.16 (DVDD), U4.2 (BASE)
- net 5v: now also J2.10, J2.20 (P20), J2.21 (P21), J2.22 (P22), J2.8, J2.9
- net 7v4: now also J24.11, J24.12, J24.13, J24.24 (P24), J24.25 (P25), Q1.10 (D_6), Q1.7 (D_3), Q1.8 (D_4), Q1.9 (D_5); no longer Q2.11 (D_7), Q2.5 (D_1), Q2.6 (D_2), Q3.11 (D_7), Q3.5 (D_1), Q3.6 (D_2)
- net GND: now also C31.1, C42.2, C43.1, C64.1, C65.2, C66.1, C68.1, C69.2, C70.1, C72.1, J2.11, J2.12, J2.13, J2.24 (P24), J2.25 (P25), J2.SH (PAD), J23.15 (P15), J23.7, J23.8, J23.SH (PAD), J24.10, J24.21 (P21), J24.22 (P22), J24.9, J24.SH (PAD), Q1.1 (S_1), Q1.2 (S_2), Q1.3 (S_3), U13.5 (AGND), U14.5 (AGND), U4.5 (AGND), Y1.2, Y1.4
- net HX711_SCK: now also U13.11 (PD_SCK), U14.11 (PD_SCK), U4.11 (PD_SCK)
- net OSC_IN: now also Y1.3
- net OSC_OUT: now also Y1.1
- net PWM_SERVO1: now also J24.1, J24.14 (P14)
- net PWM_SERVO2: now also J24.15 (P15), J24.2
- net PWM_SERVO3: now also J24.16 (P16), J24.3
- net PWM_SERVO4: now also J24.17 (P17), J24.4
- net PWM_SERVO5: now also J24.18 (P18), J24.5
- net PWM_SERVO6: now also J24.19 (P19), J24.6
- net PWM_SERVO7: now also J24.20 (P20), J24.7
- net at R2.1, U3.7 (CANH): now also J1.1 (Pin_1)
- net at R2.2, U3.6 (CANL): now also J1.2 (Pin_2)
- net at C24.1, C25.2, U9.4 (T+): now also J19.1 (+)
- net at C24.2, C26.1, U9.2 (BIAS)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: now also J19.2 (-)
- net S-1: now reaches R4.1
- net S-1: now also J23.2
- net HX711_DOUT1: now reaches U12.85 (PD4)
- net HX711_DOUT1: now also U2.12 (DOUT)
- net HX711_DOUT2: now reaches U12.86 (PD5)
- net HX711_DOUT2: now also U4.12 (DOUT)
- net HX711_DOUT3: now reaches U12.87 (PD6)
- net HX711_DOUT3: now also U13.12 (DOUT)
- net HX711_DOUT4: now reaches U12.88 (PD7)
- net HX711_DOUT4: now also U14.12 (DOUT)
- net pt6: now reaches R9.1
- net pt6: now also J2.19 (P19), J2.6
- net pt4: now reaches R17.1
- net pt4: now also J2.17 (P17), J2.4
- net at C19.1, C20.2, U7.4 (T+): now also J17.1 (+)
- net at C19.2, C21.1, U7.2 (BIAS)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: now also J17.2 (-)
- net at C14.1, C18.2, U8.4 (T+): now also J18.1 (+)
- net at C14.2, C15.1, U8.2 (BIAS)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: now also J18.2 (-)
- net pt2: now reaches R10.1
- net pt2: now also J2.15 (P15), J2.2
- net E+1: now reaches C12.1, U2.3 (AVDD), U2.4 (VFB)
- net E+1: now also J23.1
- net pt5: now reaches R1.1
- net pt5: now also J2.18 (P18), J2.5
- net pt1: now reaches R7.1
- net pt1: now also J2.1, J2.14 (P14)
- net pt3: now reaches R8.1
- net pt3: now also J2.16 (P16), J2.3
- net at R32.1, R33.2: now also Q1.4 (G)
- net S+1: now reaches R3.1
- net S+1: now also J23.9 (P9)
- net HX711_DOUT: no longer names the net of U12.18 (PC3)
- net HX711_DOUT: no longer U2.12 (DOUT)
- new net: C67.2, R25.2, U13.7 (INA-)
- new net: C44.1, R22.2, U4.8 (INA+)
- new net: C44.2, R23.2, U4.7 (INA-)
- new net: Q3.11 (D_7), Q3.5 (D_1), Q3.6 (D_2)
- new net: C67.1, R24.2, U13.8 (INA+)
- new net: C66.2, U13.6 (VBG)
- new net: Q2.11 (D_7), Q2.5 (D_1), Q2.6 (D_2)
- new net: C70.2, U14.6 (VBG)
- new net: C71.2, R27.2, U14.7 (INA-)
- new net: C71.1, R26.2, U14.8 (INA+)
- new net: Q1.11 (D_7), Q1.6 (D_2)
- new net: C43.2, U4.6 (VBG)
- new net E+2: C42.1, J23.10 (P10), U4.3 (AVDD), U4.4 (VFB)
- new net E+3: C65.1, J23.4, U13.3 (AVDD), U13.4 (VFB)
- new net E+4: C69.1, J23.13 (P13), U14.3 (AVDD), U14.4 (VFB)
- new net S+2: J23.3, R22.1
- new net S+3: J23.12 (P12), R24.1
- new net S+4: J23.6, R26.1
- new net S-2: J23.11 (P111), R23.1
- new net S-3: J23.5, R25.1
- new net S-4: J23.14 (P14), R27.1
- no-connect marks 12 -> 70
Other:
- note added: "LOAD CELL 1"
- note added: "LOAD CELL 2"
- note added: "LOAD CELL 3"
- note added: "LOAD CELL 4"
- note removed: "LOAD CELL"
- moved on the sheet: C56
