File: Ember_ECU_V0/lre_avio_daq2.kicad_pcb (KiCad board)
At the start: 2 copper layers, 4.5 x 13.4 mm, 53 parts, among them J11 USB_C_Receptacle_USB2.0_16P, J12 XT30PW-F, J13 XT30PW-F, J14 XT30PW-F, J15 XT30PW-F, J16 XT30PW-F, SW1 SW_SPDT, U1 AMS1117-5.0, U12 STM32F412VGTx, U2 HX711, U3 SN65HVD230, U5 AMS1117-5.0, U7 MAX31856, U8 MAX31856, U9 MAX31856

Commit message: erc issues and pcb related things resolved, still some remaining
Parts:
- added J3: XT60PW-M, XT60PW-M:AMASS_XT60PW-M, F.Cu at (39.9, 145.6)
- added U10: ADS8353QPWRQ1, ads8353:TSSOP16_PW_TEX-L, F.Cu at (52.5, 146.8)
- added U11: ADS8353QPWRQ1, ads8353:TSSOP16_PW_TEX-L, F.Cu at (52.5, 153.3)
- added U6: ADS8353QPWRQ1, ads8353:TSSOP16_PW_TEX-L, F.Cu at (52.5, 140.3)
- moved R6 19.4 mm to (90.2, 45.4)
- moved R7 19.4 mm to (90.2, 47.1)
- moved R17 11.2 mm to (92.6, 45.4)
- moved R18 11.2 mm to (92.6, 47.1)
- moved R19 11.2 mm to (92.6, 48.9)
- moved R20 11.2 mm to (92.6, 50.6)
- moved R21 11.2 mm to (92.6, 52.4)
- moved R3 11.2 mm to (87.7, 48.9)
- moved R4 11.2 mm to (87.7, 50.6)
- moved R5 11.2 mm to (87.7, 52.4)
- moved R30 10.2 mm to (95.1, 45.4)
- moved R31 10.2 mm to (95.1, 47.1)
- moved R32 10.2 mm to (95.1, 48.9)
- moved R33 10.2 mm to (95.1, 50.6)
- moved SW1 10.2 mm to (95.1, 52.4)
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Connections:
- U12 pad 29: /TC1_CS -> /SPI1_CS1
- U12 pad 35: /TC2_CS -> /SPI1_CS2
- U12 pad 36: /TC3_CS -> /SPI1_CS3

Commit message: ECU schematics updated
Parts:
- added C1: 1nF, Capacitor_SMD:C_0201_0603Metric, F.Cu at (193.9, 81.3)
- added C10: 10 muF, Capacitor_SMD:C_0201_0603Metric, F.Cu at (193.9, 95.3)
- added C11: 0.1 muF, Capacitor_SMD:C_0201_0603Metric, F.Cu at (193.9, 97.0)
- added C12: 10 muF, Capacitor_SMD:C_0201_0603Metric, F.Cu at (196.3, 81.3)
- added C13: 0.1 muF, Capacitor_SMD:C_0201_0603Metric, F.Cu at (196.3, 83.0)
- added C14: 0.1 muF, Capacitor_SMD:C_0201_0603Metric, F.Cu at (196.3, 84.8)
- added C15: 0.01 muF, Capacitor_SMD:C_0201_0603Metric, F.Cu at (196.3, 86.5)
- added C16: 0.1 muF, Capacitor_SMD:C_0201_0603Metric, F.Cu at (196.3, 88.3)
- added C17: 0.1 muF, Capacitor_SMD:C_0201_0603Metric, F.Cu at (196.3, 90.0)
- added C18: 0.01 muF, Capacitor_SMD:C_0201_0603Metric, F.Cu at (196.3, 91.8)
- added C19: 0.1 muF, Capacitor_SMD:C_0201_0603Metric, F.Cu at (196.3, 93.5)
- added C2: 1nF, Capacitor_SMD:C_0201_0603Metric, F.Cu at (193.9, 83.0)
- added C20: 0.01 muF, Capacitor_SMD:C_0201_0603Metric, F.Cu at (196.3, 95.3)
- added C21: 0.01 muF, Capacitor_SMD:C_0201_0603Metric, F.Cu at (196.3, 97.0)
- added C22: 0.1 muF, Capacitor_SMD:C_0201_0603Metric, F.Cu at (198.8, 81.3)
- added C23: 0.1 muF, Capacitor_SMD:C_0201_0603Metric, F.Cu at (198.8, 83.0)
- added C24: 0.1 muF, Capacitor_SMD:C_0201_0603Metric, F.Cu at (198.8, 84.8)
- added C25: 0.01 muF, Capacitor_SMD:C_0201_0603Metric, F.Cu at (198.8, 86.5)
- added C26: 0.01 muF, Capacitor_SMD:C_0201_0603Metric, F.Cu at (198.8, 88.3)
- added C27: 0.1 muF, Capacitor_SMD:C_0201_0603Metric, F.Cu at (198.8, 90.0)
- added C28: 0.1 muF, Capacitor_SMD:C_0201_0603Metric, F.Cu at (198.8, 91.8)
- added C3: 1nF, Capacitor_SMD:C_0201_0603Metric, F.Cu at (193.9, 84.8)
- added C30: C, Capacitor_SMD:C_0201_0603Metric, F.Cu at (198.8, 93.5)
- added C31: 10 muF, Capacitor_SMD:C_0201_0603Metric, F.Cu at (198.8, 95.3)
- added C35: C, Capacitor_SMD:C_0201_0603Metric, F.Cu at (198.8, 97.0)
- added C39: C, Capacitor_SMD:C_0201_0603Metric, F.Cu at (201.2, 81.3)
- added C4: 1nF, Capacitor_SMD:C_0201_0603Metric, F.Cu at (193.9, 86.5)
- added C42: 10 muF, Capacitor_SMD:C_0201_0603Metric, F.Cu at (201.2, 83.0)
- added C43: 0.1 muF, Capacitor_SMD:C_0201_0603Metric, F.Cu at (201.2, 84.8)
- added C44: 0.1 muF, Capacitor_SMD:C_0201_0603Metric, F.Cu at (201.2, 86.5)
- added C45: 100 nF, Capacitor_SMD:C_0201_0603Metric, F.Cu at (201.2, 88.3)
- added C46: 1 muF, Capacitor_SMD:C_0201_0603Metric, F.Cu at (201.2, 90.0)
- added C47: 100 nF, Capacitor_SMD:C_0201_0603Metric, F.Cu at (201.2, 91.8)
- added C48: 1 muF, Capacitor_SMD:C_0201_0603Metric, F.Cu at (201.2, 93.5)
- added C49: 1 muF, Capacitor_SMD:C_0201_0603Metric, F.Cu at (201.2, 95.3)
- added C5: 1nF, Capacitor_SMD:C_0201_0603Metric, F.Cu at (193.9, 88.3)
- added C50: 100 nF, Capacitor_SMD:C_0201_0603Metric, F.Cu at (201.2, 97.0)
- added C51: 100 nF, Capacitor_SMD:C_0201_0603Metric, F.Cu at (203.7, 81.3)
- added C52: 1 muF, Capacitor_SMD:C_0201_0603Metric, F.Cu at (203.7, 83.0)
- added C53: 100 nF, Capacitor_SMD:C_0201_0603Metric, F.Cu at (203.7, 84.8)
- added C54: 100 nF, Capacitor_SMD:C_0201_0603Metric, F.Cu at (203.7, 86.5)
- added C55: 100 nF, Capacitor_SMD:C_0201_0603Metric, F.Cu at (203.7, 88.3)
- added C56: 100 nF, Capacitor_SMD:C_0201_0603Metric, F.Cu at (203.7, 90.0)
- added C57: 100 nF, Capacitor_SMD:C_0201_0603Metric, F.Cu at (203.7, 91.8)
- added C58: 100 nF, Capacitor_SMD:C_0201_0603Metric, F.Cu at (203.7, 93.5)
- added C59: 10 nF, Capacitor_SMD:C_0201_0603Metric, F.Cu at (203.7, 95.3)
- added C6: 1nF, Capacitor_SMD:C_0201_0603Metric, F.Cu at (193.9, 90.0)
- added C60: 1 muF, Capacitor_SMD:C_0201_0603Metric, F.Cu at (203.7, 97.0)
- added C61: 100 nF, Capacitor_SMD:C_0201_0603Metric, F.Cu at (206.1, 81.3)
- added C62: 4.7 muF, Capacitor_SMD:C_0201_0603Metric, F.Cu at (206.1, 83.0)
- added C63: 4.7 muF, Capacitor_SMD:C_0201_0603Metric, F.Cu at (206.1, 84.8)
- added C64: 10 muF, Capacitor_SMD:C_0201_0603Metric, F.Cu at (206.1, 86.5)
- added C65: 10 muF, Capacitor_SMD:C_0201_0603Metric, F.Cu at (206.1, 88.3)
- added C66: 0.1 muF, Capacitor_SMD:C_0201_0603Metric, F.Cu at (206.1, 90.0)
- added C67: 0.1 muF, Capacitor_SMD:C_0201_0603Metric, F.Cu at (206.1, 91.8)
- added C68: 10 muF, Capacitor_SMD:C_0201_0603Metric, F.Cu at (206.1, 93.5)
- added C69: 10 muF, Capacitor_SMD:C_0201_0603Metric, F.Cu at (206.1, 95.3)
- added C70: 0.1 muF, Capacitor_SMD:C_0201_0603Metric, F.Cu at (206.1, 97.0)
- added C71: 0.1 muF, Capacitor_SMD:C_0201_0603Metric, F.Cu at (208.6, 81.3)
- added C72: 100 nF, Capacitor_SMD:C_0201_0603Metric, F.Cu at (208.6, 83.0)
- added C8: 20 pF, Capacitor_SMD:C_0201_0603Metric, F.Cu at (193.9, 91.8)
- added C9: 20 pF, Capacitor_SMD:C_0201_0603Metric, F.Cu at (193.9, 93.5)
- added D1: D_Schottky, RSX501LAM20TR:DIO_RB050LAM_ROM, F.Cu at (58.9, 170.6)
- added D2: D_Schottky, RSX501LAM20TR:DIO_RB050LAM_ROM, F.Cu at (58.9, 174.7)
- added J1: Conn_01x02_Socket, Connector_JST:JST_EH_B2B-EH-A_1x02_P2.50mm_Vertical, F.Cu at (163.8, 37.3)
- added J10: Conn_01x03_Socket, Connector_AMASS:AMASS_MR30PW-FB_1x03_P3.50mm_Horizontal, F.Cu at (233.5, 77.9)
- added J17: SMPW-CC-K-M, SMPW-CC-K-M:SMPWCCKM, F.Cu at (139.1, 86.5)
- added J18: SMPW-CC-K-M, SMPW-CC-K-M:SMPWCCKM, F.Cu at (150.2, 86.5)
- added J19: SMPW-CC-K-M, SMPW-CC-K-M:SMPWCCKM, F.Cu at (161.3, 86.5)
- added J2: DB25_Socket_MountingHoles, Connector_Dsub:DSUB-25_Socket_Horizontal_P2.77x2.84mm_EdgePinOffset4.94mm_Housed_MountingHolesOffset4.94mm, F.Cu at (60.8, 51.4)
- added J23: DA15_Socket_MountingHoles, Connector_Dsub:DSUB-15_Socket_Horizontal_P2.77x2.84mm_EdgePinOffset4.94mm_Housed_MountingHolesOffset4.94mm, F.Cu at (149.3, 38.0)
- added J24: DB25_Socket_MountingHoles, Connector_Dsub:DSUB-25_Socket_Horizontal_P2.77x2.84mm_EdgePinOffset4.94mm_Housed_MountingHolesOffset4.94mm, F.Cu at (163.2, 19.3)
- added J5: Conn_01x03_Socket, Connector_AMASS:AMASS_MR30PW-FB_1x03_P3.50mm_Horizontal, F.Cu at (146.2, 77.9)
- added J6: Conn_01x03_Socket, Connector_AMASS:AMASS_MR30PW-FB_1x03_P3.50mm_Horizontal, F.Cu at (163.7, 77.9)
- added J7: Conn_01x03_Socket, Connector_AMASS:AMASS_MR30PW-FB_1x03_P3.50mm_Horizontal, F.Cu at (181.1, 77.9)
- added J8: Conn_01x03_Socket, Connector_AMASS:AMASS_MR30PW-FB_1x03_P3.50mm_Horizontal, F.Cu at (198.6, 77.9)
- added J9: Conn_01x03_Socket, Connector_AMASS:AMASS_MR30PW-FB_1x03_P3.50mm_Horizontal, F.Cu at (216.0, 77.9)
- added Q1: SISA96DN-T1-GE3, SISA96DN-T1-GE3:SIS862DNT1GE3, F.Cu at (132.4, 148.3)
- added Q2: SISA96DN-T1-GE3, SISA96DN-T1-GE3:SIS862DNT1GE3, F.Cu at (132.4, 154.4)
- added Q3: SISA96DN-T1-GE3, SISA96DN-T1-GE3:SIS862DNT1GE3, F.Cu at (132.4, 160.6)
- added R22: 100, Resistor_SMD:R_0201_0603Metric, F.Cu at (208.6, 84.8)
- added R23: 100, Resistor_SMD:R_0201_0603Metric, F.Cu at (208.6, 86.5)
- added R24: 100, Resistor_SMD:R_0201_0603Metric, F.Cu at (208.6, 88.3)
- added R25: 100, Resistor_SMD:R_0201_0603Metric, F.Cu at (208.6, 90.0)
- added R26: 100, Resistor_SMD:R_0201_0603Metric, F.Cu at (208.6, 91.8)
- added R27: 100, Resistor_SMD:R_0201_0603Metric, F.Cu at (208.6, 93.5)
- added U13: HX711, Package_SO:SOIC-16_3.9x9.9mm_P1.27mm, F.Cu at (180.0, 86.3)
- added U14: HX711, Package_SO:SOIC-16_3.9x9.9mm_P1.27mm, F.Cu at (188.4, 86.3)
- added U4: HX711, Package_SO:SOIC-16_3.9x9.9mm_P1.27mm, F.Cu at (171.5, 86.3)
- added Y1: Crystal_8Mhz, Crystal:Crystal_SMD_7050-4Pin_7.0x5.0mm, F.Cu at (214.6, 83.9)
- SW1: footprint Resistor_SMD:R_0201_0603Metric -> Button_Switch_SMD:SW_SPDT_PCM12
Connections:
- net Net-(J2-Pin_1) renamed /E+1
- C33 pad 1: 3v3 -> /3v3
- C37 pad 1: 3v3 -> /3v3
- C41 pad 1: 3v3 -> /3v3
- R1 pad 1: Net-(J5-Pin_2) -> /pt5
- R10 pad 1: Net-(J9-Pin_2) -> /pt2
- R11 pad 1: 3v3 -> /3v3
- R12 pad 1: 3v3 -> /3v3
- R13 pad 1: 3v3 -> /3v3
- R14 pad 1: 3v3 -> /3v3
- R15 pad 1: +3.3V -> /3v3
- R16 pad 1: +3.3V -> /3v3
- R17 pad 1: Net-(J10-Pin_2) -> /pt4
- R3 pad 1: Net-(J2-Pin_3) -> /S+1
- R4 pad 1: Net-(J2-Pin_4) -> /S-1
- R7 pad 1: Net-(J6-Pin_2) -> /pt1
- R8 pad 1: Net-(J7-Pin_2) -> /pt3
- R9 pad 1: Net-(J8-Pin_2) -> /pt6
- U10 pad 9: 3v3 -> /3v3
- U11 pad 9: 3v3 -> /3v3
- U12 pad 100: 3v3 -> /3v3
- U12 pad 11: 3v3 -> /3v3
- U12 pad 18: /HX711_DOUT -> unconnected-(U12-PC3-Pad18)
- U12 pad 19: 3v3 -> /3v3
- U12 pad 22: unconnected-(U12-VDDA-Pad22) -> /3v3
- U12 pad 28: 3v3 -> /3v3
- U12 pad 29: /SPI1_CS1 -> /TC1_CS
- U12 pad 35: /SPI1_CS2 -> /TC2_CS
- U12 pad 36: /SPI1_CS3 -> /TC3_CS
- U12 pad 50: 3v3 -> /3v3
- U12 pad 6: 3v3 -> /3v3
- U12 pad 75: 3v3 -> /3v3
- U12 pad 85: unconnected-(U12-PD4-Pad85) -> /HX711_DOUT1
- U12 pad 86: unconnected-(U12-PD5-Pad86) -> /HX711_DOUT2
- U12 pad 87: unconnected-(U12-PD6-Pad87) -> /HX711_DOUT3
- U12 pad 88: unconnected-(U12-PD7-Pad88) -> /HX711_DOUT4
- U2 pad 1: 3v3 -> /3v3
- U2 pad 12: /HX711_DOUT -> /HX711_DOUT1
- U2 pad 15: 3v3 -> /3v3
- U2 pad 16: 3v3 -> /3v3
- U2 pad 2: 3v3 -> /3v3
- U3 pad 3: 3v3 -> /3v3
- U5 pad 2: 3v3 -> /3v3
- U6 pad 9: 3v3 -> /3v3
- U7 pad 5: 3v3 -> /3v3
- U7 pad 8: 3v3 -> /3v3
- U8 pad 5: 3v3 -> /3v3
- U8 pad 8: 3v3 -> /3v3
- U9 pad 5: +3.3V -> /3v3
- U9 pad 8: +3.3V -> /3v3
Routing:
- net /3v3: track 0.00 -> 128.5 mm, vias 0 -> 8
- net 3v3: track 108.2 -> 0.00 mm, vias 4 -> 0
- net +3.3V: track 20.4 -> 0.00 mm, vias 4 -> 0
- net /HX711_DOUT: track 20.3 -> 0.00 mm
- net (no net): track 0.00 -> 20.3 mm

Commit message: commit
Parts:
- removed D1, D2: D_Schottky, RSX501LAM20TR:DIO_RB050LAM_ROM
- removed J10, J5, J6, J7, J8, J9: Conn_01x03_Socket, Connector_AMASS:AMASS_MR30PW-FB_1x03_P3.50mm_Horizontal
- removed J17, J18, J19: SMPW-CC-K-M, SMPW-CC-K-M:SMPWCCKM
- removed J3: XT60PW-M, XT60PW-M:AMASS_XT60PW-M
- removed Q1, Q2, Q3: SISA96DN-T1-GE3, SISA96DN-T1-GE3:SIS862DNT1GE3
- added D3: LED, LED_SMD:LED_0603_1608Metric, F.Cu at (56.7, 48.7)
- added LS1: CMT-8530S-SMT, CMT-8530S-SMT:CUI_CMT-8530S-SMT, F.Cu at (155.4, 111.4)
- added Q5: ~, CJ3400:SOT95P240X115-3N, F.Cu at (165.0, 105.1)
- added R34: R, Resistor_SMD:R_0603_1608Metric, F.Cu at (35.3, 73.6)
- added R35: 100, Resistor_SMD:R_0603_1608Metric, F.Cu at (35.3, 76.1)
- added R36: 10k, Resistor_SMD:R_0603_1608Metric, F.Cu at (35.3, 78.6)
- added U15: WS2812B-2020, footprints:SMT_12B-2020_WDS, F.Cu at (57.0, 38.3)
- added U16: WS2812B-2020, footprints:SMT_12B-2020_WDS, F.Cu at (57.0, 42.0)
- added U17: WS2812B-2020, footprints:SMT_12B-2020_WDS, F.Cu at (57.0, 45.6)
- moved C72 156.9 mm to (54.2, 54.6)
- moved C71 156.8 mm to (51.8, 77.3)
- moved C30 156.8 mm to (46.9, 54.6)
- moved C31 156.8 mm to (46.9, 56.3)
- moved C58 156.8 mm to (51.8, 54.6)
- moved C59 156.8 mm to (51.8, 56.3)
- moved C60 156.8 mm to (51.8, 58.1)
- moved C61 155.8 mm to (51.8, 59.8)
- moved C62 155.8 mm to (51.8, 61.6)
- moved C63 155.8 mm to (51.8, 63.3)
- moved C64 155.8 mm to (51.8, 65.1)
- moved C65 155.8 mm to (51.8, 66.8)
- moved C66 155.8 mm to (51.8, 68.6)
- moved C67 155.8 mm to (51.8, 70.3)
- moved C68 155.8 mm to (51.8, 72.1)
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Connections:
- U12 pad 8: unconnected-(U12-PC14-Pad8) -> /Buzzer_G
- U12 pad 9: unconnected-(U12-PC15-Pad9) -> /DI1
Routing:
- net /HX711_SCK: track 7.14 -> 63.5 mm
- net (no net): track 20.3 -> 73.3 mm
- net /3v3: track 128.5 -> 79.0 mm, vias 8 -> 6
- net Net-(U13-INA-): track 0.00 -> 38.4 mm, vias 0 -> 2
- net /S-4: track 0.00 -> 36.5 mm
- net /SPI1_MOSI: track 34.2 -> 0.00 mm, vias 6 -> 0
- net /SPI1_SCK: track 32.8 -> 0.00 mm, vias 4 -> 0
- net GND: track 149.7 -> 117.3 mm, vias 4 -> 0
- net /S-3: track 0.00 -> 32.2 mm
- net /SPI1_MISO: track 31.7 -> 0.00 mm, vias 6 -> 0
- net /S+4: track 0.00 -> 31.2 mm
- net Net-(U14-INA+): track 0.00 -> 30.5 mm
- net Net-(U14-INA-): track 0.00 -> 30.1 mm
- net /HX711_DOUT2: track 0.00 -> 24.6 mm, vias 0 -> 2
- net /HX711_DOUT4: track 0.00 -> 24.4 mm, vias 0 -> 2
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Other:
- outline, holes or cut-outs redrawn

Commit message: half routed ECU
Parts:
- added C7: 47 uF, Capacitor_SMD:C_0603_1608Metric, F.Cu at (78.6, 123.7)
- added C73: 47 uF, Capacitor_SMD:C_0603_1608Metric, F.Cu at (77.9, 108.4)
- added C74: C, Capacitor_SMD:C_0603_1608Metric, F.Cu at (77.9, 110.9)
- added C75: 47 uF, Capacitor_SMD:C_0603_1608Metric, F.Cu at (77.9, 113.4)
- added C76: 47 uF, Capacitor_SMD:C_0603_1608Metric, F.Cu at (78.6, 126.2)
- added D1: D_Schottky, RSX501LAM20TR:DIO_RB050LAM_ROM, F.Cu at (72.6, 150.4)
- added D2: D_Schottky, RSX501LAM20TR:DIO_RB050LAM_ROM, F.Cu at (72.6, 154.6)
- added D4: ESDCAN02-2BWY, ESDCAN02-2BWY:SOT65P210X110-3N, F.Cu at (78.4, 150.2)
- added D5: ESDCAN02-2BWY, ESDCAN02-2BWY:SOT65P210X110-3N, F.Cu at (78.4, 154.0)
- added J17: SMPW-CC-K-M, SMPW-CC-K-M:SMPWCCKM, F.Cu at (48.4, 128.4)
- added J18: SMPW-CC-K-M, SMPW-CC-K-M:SMPWCCKM, F.Cu at (59.5, 128.4)
- added J19: SMPW-CC-K-M, SMPW-CC-K-M:SMPWCCKM, F.Cu at (70.6, 128.4)
- added J3: XT60PW-M, XT60PW-M:AMASS_XT60PW-M, F.Cu at (53.7, 151.1)
- added J4: Conn_01x02_Socket, Connector_JST:JST_EH_B2B-EH-A_1x02_P2.50mm_Vertical, F.Cu at (72.7, 145.1)
- added Q1: SISA96DN-T1-GE3, SISA96DN-T1-GE3:SIS862DNT1GE3, F.Cu at (65.8, 145.6)
- added Q2: SISA96DN-T1-GE3, SISA96DN-T1-GE3:SIS862DNT1GE3, F.Cu at (65.8, 151.7)
- added Q3: SISA96DN-T1-GE3, SISA96DN-T1-GE3:SIS862DNT1GE3, F.Cu at (65.8, 157.9)
- added R2: R, Resistor_SMD:R_0603_1608Metric, F.Cu at (78.6, 128.7)
- added R37: R, Resistor_SMD:R_0603_1608Metric, F.Cu at (77.9, 115.9)
- added R38: 10k, Resistor_SMD:R_0603_1608Metric, F.Cu at (198.8, 121.5)
- added R39: 10k, Resistor_SMD:R_0603_1608Metric, F.Cu at (203.0, 105.3)
- added R40: 10k, Resistor_SMD:R_0603_1608Metric, F.Cu at (210.0, 121.5)
- C1, C10, C11, C12, C13, C14, C15, C16, C17, C18, C19, C2, C20, C21, C22, C23, C24, C25, C26, C27, C28, C29, C3, C30, C31, C32, C33, C34, C35, C36, C37, C38, C39, C4, C40, C41, C42, C43, C44, C45, C46, C47, C48, C49, C5, C50, C51, C52, C53, C54, C55, C56, C57, C58, C59, C6, C60, C61, C62, C63, C64, C65, C66, C67, C68, C69, C70, C71, C72, C8, C9: footprint Capacitor_SMD:C_0201_0603Metric -> Capacitor_SMD:C_0603_1608Metric
- R1, R10, R11, R12, R13, R14, R15, R16, R17, R18, R19, R20, R21, R22, R23, R24, R25, R26, R27, R28, R29, R3, R30, R31, R32, R33, R4, R5, R6, R7, R8, R9: footprint Resistor_SMD:R_0201_0603Metric -> Resistor_SMD:R_0603_1608Metric
- moved C30 181.6 mm to (210.8, 132.8), turned to 90 degrees
- moved C58 180.8 mm to (228.3, 93.4)
- moved C63 179.3 mm to (228.3, 95.0)
- moved C54 178.5 mm to (223.5, 110.9), turned to -90 degrees
- moved C33 177.3 mm to (213.1, 121.5)
- moved C62 177.2 mm to (222.0, 110.9), turned to -90 degrees
- moved C5 174.6 mm to (201.8, 131.9)
- moved C29 173.8 mm to (209.2, 132.8), turned to 90 degrees
- moved C32 172.0 mm to (206.8, 121.5)
- moved R1 171.0 mm to (206.7, 133.6)
- moved C6 168.7 mm to (202.3, 116.0)
- moved C35 167.6 mm to (199.4, 132.7), turned to 90 degrees
- moved C55 166.9 mm to (212.1, 110.9), turned to -90 degrees
- moved C34 166.7 mm to (197.7, 132.7), turned to 90 degrees
- moved C37 164.4 mm to (201.9, 121.5)
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Connections:
- J1 pad 1: Net-(J1-Pin_1) -> /CAN_H
- J1 pad 2: Net-(J1-Pin_2) -> /CAN_L
- R1 pad 1: /pt5 -> /pt1
- R10 pad 1: /pt2 -> /pt4
- R17 pad 1: /pt4 -> /pt6
- R7 pad 1: /pt1 -> /pt3
- R8 pad 1: /pt3 -> /pt5
- R9 pad 1: /pt6 -> /pt2
- U3 pad 6: Net-(J1-Pin_2) -> /CAN_L
- U3 pad 7: Net-(J1-Pin_1) -> /CAN_H
Routing:
- net GND: track 117.3 -> 0.00 mm
- net /7v4: track 90.4 -> 0.00 mm
- net (no net): track 73.3 -> 0.00 mm
- net /HX711_SCK: track 63.5 -> 0.00 mm
- net /SPI3_SCK: track 0.00 -> 55.0 mm, vias 0 -> 2
- net /SPI3_MISO: track 0.00 -> 53.4 mm, vias 0 -> 2
- net /SPI3_MOSI: track 0.00 -> 51.8 mm, vias 0 -> 2
- net /pt2: track 0.00 -> 42.3 mm
- net /3v3: track 79.0 -> 37.9 mm, vias 6 -> 4
- net Net-(U13-INA-): track 38.4 -> 0.00 mm
- net /S-4: track 36.5 -> 0.00 mm
- net /S-3: track 32.2 -> 0.00 mm
- net /S+4: track 31.2 -> 0.00 mm
- net Net-(U14-INA+): track 30.5 -> 0.00 mm
- net Net-(U14-INA-): track 30.1 -> 0.00 mm
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Other:
- copper layers 2 -> 4

Commit message: commit
Parts:
- moved C16 199.8 mm to (229.4, 130.0), turned to 180 degrees
- moved C18 199.0 mm to (229.4, 131.5), turned to 180 degrees
- moved C15 196.1 mm to (229.5, 134.8), turned to 180 degrees
- moved C14 196.0 mm to (229.4, 133.1), turned to 180 degrees
- moved C19 189.5 mm to (211.7, 148.9), turned to 90 degrees
- moved C22 189.4 mm to (214.0, 149.4), turned to 90 degrees
- moved C17 188.7 mm to (218.5, 129.1)
- moved R11 183.5 mm to (229.4, 128.5), turned to 180 degrees
- moved C21 179.6 mm to (208.4, 136.6)
- moved J18 178.0 mm to (237.4, 135.3), turned to 180 degrees
- moved R14 176.5 mm to (212.5, 137.4), turned to -90 degrees
- moved C71 176.5 mm to (227.5, 60.9), turned to 90 degrees
- moved C68 176.0 mm to (226.8, 53.5)
- moved C69 175.9 mm to (226.8, 56.1)
- moved C70 175.8 mm to (226.7, 58.6)
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Routing:
- net GND: track 0.00 -> 265.5 mm, vias 0 -> 6
- net /3v3: track 37.9 -> 213.6 mm, vias 4 -> 6
- net /7v4: track 0.00 -> 106.0 mm
- net (no net): track 0.00 -> 78.7 mm
- net /5v: track 24.1 -> 93.7 mm
- net /SPI1_MISO: track 0.00 -> 66.5 mm, vias 0 -> 5
- net /SPI1_SCK: track 0.00 -> 65.7 mm, vias 0 -> 4
- net /SPI1_MOSI: track 0.00 -> 62.0 mm, vias 0 -> 6
- net /HX711_SCK: track 0.00 -> 44.1 mm
- net /Buzzer_G: track 0.00 -> 39.2 mm, vias 0 -> 4
- net /PWM_SERVO7: track 0.00 -> 39.2 mm
- net /HX711_DOUT2: track 0.00 -> 39.1 mm
- net /PWM_SERVO6: track 0.00 -> 34.6 mm
- net Net-(J19--): track 0.00 -> 33.3 mm
- net /PWM_SERVO5: track 0.00 -> 30.9 mm
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
Commit message: commit
Parts:
- moved Q1 134.1 mm to (160.0, 50.2), turned to 90 degrees
- moved Q2 119.6 mm to (129.5, 50.5), turned to 90 degrees
- moved R29 109.3 mm to (129.5, 57.9)
- moved R28 73.3 mm to (131.2, 55.4)
- moved Q3 72.5 mm to (145.0, 49.8)
- moved R30 72.5 mm to (148.6, 50.4)
- moved R31 72.5 mm to (151.5, 51.2)
- moved R20 64.9 mm to (121.2, 58.3)
- moved R19 54.2 mm to (108.9, 48.6)
- moved R32 54.2 mm to (161.7, 54.2)
- moved R33 54.0 mm to (160.1, 56.5)
- moved R18 50.4 mm to (105.4, 48.6)
Routing:
- net /7v4: track 106.0 -> 121.4 mm
- net GND: track 265.5 -> 280.4 mm
- net Net-(Q2-G): track 0.00 -> 5.97 mm
- net Net-(Q1-G): track 0.00 -> 4.90 mm
- net /BATTERY_MON: track 0.00 -> 1.88 mm
- net /HX711_DOUT3: vias 2 -> 1
- net /HX711_DOUT2: vias 2 -> 1
- net /HX711_DOUT1: vias 4 -> 2
- net /3v3: vias 6 -> 3

Commit message: commit
Parts:
- removed the R2 at (54.2, 58.1)
- moved R21 191.8 mm to (239.8, 124.0)
- moved J1 185.6 mm to (246.6, 131.8), turned to -90 degrees
- moved D3 178.5 mm to (213.7, 163.8), turned to 180 degrees
- moved R34 178.4 mm to (213.8, 165.9), turned to 180 degrees
- moved J4 177.3 mm to (249.9, 145.0), turned to 90 degrees
- moved U15 173.1 mm to (211.8, 115.8), turned to -90 degrees
- moved C20 172.9 mm to (190.2, 154.5), turned to 90 degrees
- moved R5 171.8 mm to (210.3, 163.8), turned to 180 degrees
- moved C75 171.0 mm to (245.7, 146.4)
- moved U16 169.4 mm to (211.7, 111.2), turned to -90 degrees
- moved J3 168.7 mm to (207.6, 154.4), turned to 180 degrees
- moved C48 168.7 mm to (209.4, 114.7), turned to 90 degrees
- moved C76 168.0 mm to (245.8, 142.5), turned to 180 degrees
- moved C47 167.6 mm to (207.6, 114.8), turned to 90 degrees
- moved C31 166.5 mm to (213.4, 53.1)
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Routing:
- net GND: track 280.4 -> 543.1 mm, vias 6 -> 24
- net /DI1: track 0.00 -> 180.9 mm, vias 0 -> 4
- net /5v: track 93.7 -> 213.2 mm, vias 0 -> 4
- net /ARM: track 0.00 -> 115.3 mm, vias 0 -> 2
- net /BATTERY_MON: track 1.88 -> 111.3 mm, vias 0 -> 2
- net /PWM_SERVO5: track 30.9 -> 126.6 mm, vias 0 -> 2
- net /7v4: track 121.4 -> 215.2 mm
- net /CAN_H: track 0.00 -> 90.1 mm, vias 0 -> 4
- net /CAN_L: track 0.00 -> 84.3 mm, vias 0 -> 5
- net /Conn1: track 0.00 -> 78.3 mm, vias 0 -> 2
- net /PWM_SERVO3: track 3.41 -> 80.3 mm, vias 0 -> 2
- net /ADS2_CS: track 3.13 -> 79.1 mm, vias 0 -> 2
- net (no net): track 78.7 -> 7.00 mm
- net /PWM_SERVO2: track 3.41 -> 71.5 mm, vias 0 -> 2
- net /Conn2: track 0.00 -> 60.6 mm
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Other:
- outline, holes or cut-outs redrawn

Commit message: Added the PDB
Parts:
- moved D1 13.1 mm to (153.6, 123.7), turned to 180 degrees
Routing:
- net /5v: track 213.2 -> 197.6 mm
- net Net-(D1-A): track 9.05 -> 20.0 mm
- net GND: track 543.1 -> 541.3 mm
