File: Ember_ECU_V0/lre_avio_daq2.kicad_pcb (KiCad board)
At the start: 4 copper layers, 4.5 x 13.4 mm, 162 parts, among them J1 Conn_01x02_Socket, J11 USB_C_Receptacle_USB2.0_16P, J12 XT30PW-F, J13 XT30PW-F, J14 XT30PW-F, J15 XT30PW-F, J16 XT30PW-F, J17 SMPW-CC-K-M, J18 SMPW-CC-K-M, J19 SMPW-CC-K-M, J2 DB25_Socket_MountingHoles, J23 DA15_Socket_MountingHoles, J24 DB25_Socket_MountingHoles, J3 XT60PW-M, J4 Conn_01x02_Socket, Q1 SISA96DN-T1-GE3, Q2 SISA96DN-T1-GE3, Q3 SISA96DN-T1-GE3, SW1 SW_SPDT, U1 AMS1117-5.0, U10 ADS8353QPWRQ1, U11 ADS8353QPWRQ1, U12 STM32F412VGTx, U13 HX711, U14 HX711, U15 WS2812B-2020, U16 WS2812B-2020, U17 WS2812B-2020, U2 HX711, U3 SN65HVD230, U4 HX711, U5 AMS1117-5.0, U6 ADS8353QPWRQ1, U7 MAX31856, U8 MAX31856, U9 MAX31856, Y1 Crystal_8Mhz

Commit message: made changes to the pcb and fixed the schematic for can and add footptints
Parts:
- removed U3: SN65HVD230, Package_SO:SOIC-8_3.9x4.9mm_P1.27mm
- added C77: 47pf, Capacitor_SMD:C_0603_1608Metric, F.Cu at (128.1, 101.8)
- added C78: 47pf, Capacitor_SMD:C_0603_1608Metric, F.Cu at (128.2, 98.8)
- added C79: 47pf, Capacitor_SMD:C_0603_1608Metric, F.Cu at (127.1, 112.7)
- added C80: 47pf, Capacitor_SMD:C_0603_1608Metric, F.Cu at (127.1, 115.2)
- added C81: 100nF, Capacitor_SMD:C_0603_1608Metric, F.Cu at (26.9, 94.0)
- added J10: Conn_01x02_Pin, Connector_JST:JST_EH_B2B-EH-A_1x02_P2.50mm_Vertical, F.Cu at (132.4, 123.0)
- added J20: Conn_01x02_Pin, Connector_JST:JST_EH_B2B-EH-A_1x02_P2.50mm_Vertical, F.Cu at (132.5, 133.8)
- added R41: 10K, Resistor_SMD:R_0603_1608Metric, B.Cu at (224.1, 94.0)
- added R42: 10K, Resistor_SMD:R_0603_1608Metric, B.Cu at (207.5, 94.0)
- added R43: 10K, Resistor_SMD:R_0603_1608Metric, B.Cu at (216.3, 94.0)
- added U18: TCAN330, Package_SO:SOIC-8_3.9x4.9mm_P1.27mm, F.Cu at (230.1, 76.6)
- C10, C11, C12, C13, C14, C15, C16, C17, C18, C19, C20, C21, C22, C23, C24, C25, C26, C27, C28, C31, C41, C42, C43, C44, C6, C64, C65, C66, C67, C68, C69, C70, C71, R11, R12, R13, R14, R15, R16, R17, R22, R23, R24, R25, R26, R27, R3, R4, U13, U14, U2, U4, U7, U8, U9: moved to B.Cu
- D1, D2: footprint RSX501LAM20TR:DIO_RB050LAM_ROM -> Diode_SMD:D_2114_3652Metric
- Q1, Q2, Q3: footprint SISA96DN-T1-GE3:SIS862DNT1GE3 -> footprints:MOSFET_1DN-T1-GE3_VIS
- R2: footprint Resistor_SMD:R_0603_1608Metric -> Resistor_SMD:R_0603_1608Metric_Pad0.98x0.95mm_HandSolder
- U15, U16, U17: footprint footprints:SMT_12B-2020_WDS -> ggg:SMT_12B-2020_WDS
- moved C76 189.2 mm to (91.4, 33.1), turned to 0 degrees
- moved U17 186.7 mm to (25.2, 119.5), turned to 0 degrees
- moved U15 186.6 mm to (25.2, 112.1), turned to 0 degrees
- moved U16 186.5 mm to (25.2, 115.8), turned to 0 degrees
- moved J3 184.1 mm to (25.9, 183.9), turned to 0 degrees
- moved C75 176.5 mm to (87.4, 68.3)
- moved R19 173.8 mm to (95.4, 40.7)
- moved D3 173.8 mm to (67.1, 70.5), turned to 0 degrees
- moved R18 172.4 mm to (95.4, 38.2)
- moved J4 169.6 mm to (105.0, 57.0), turned to 0 degrees
- moved R34 169.5 mm to (99.4, 40.7), turned to 0 degrees
- moved R5 167.0 mm to (44.0, 178.6), turned to 0 degrees
- moved D5 165.7 mm to (45.0, 117.9)
- moved D4 165.6 mm to (45.0, 114.1)
- moved R21 164.2 mm to (95.4, 45.7)
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Connections:
- U12 pad 70: /CAN1_RX -> /CAN_RX
- U12 pad 71: /CAN1_TX -> /CAN_TX
- U7 pad 9: /SPI1_CS1 -> /TC1_CS
- U8 pad 9: /SPI1_CS2 -> /TC2_CS
- U9 pad 9: /SPI1_CS3 -> /TC3_CS
Routing:
- net GND: track 543.1 -> 31.9 mm, vias 24 -> 0
- net /3v3: track 274.0 -> 79.1 mm, vias 6 -> 1
- net /DI1: track 180.9 -> 0.00 mm, vias 4 -> 0
- net /5v: track 213.2 -> 41.4 mm, vias 4 -> 0
- net /7v4: track 215.2 -> 76.9 mm
- net /PWM_SERVO5: track 126.6 -> 0.00 mm, vias 2 -> 0
- net /ARM: track 115.3 -> 0.00 mm, vias 2 -> 0
- net /BATTERY_MON: track 111.3 -> 0.00 mm, vias 2 -> 0
- net /CAN_H: track 90.1 -> 0.00 mm, vias 4 -> 0
- net /CAN_L: track 84.3 -> 0.00 mm, vias 5 -> 0
- net /PWM_SERVO3: track 80.3 -> 0.00 mm, vias 2 -> 0
- net /Conn1: track 78.3 -> 0.00 mm, vias 2 -> 0
- net /PWM_SERVO2: track 71.5 -> 0.00 mm, vias 2 -> 0
- net /ADS2_CS: track 79.1 -> 14.1 mm
- net /Conn2: track 60.6 -> 0.00 mm
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Other:
- board size 4.5 x 13.4 mm -> 13.4 x 4.5 mm
