File: Ember_ECU_V0/_restore_backup_2026-09-24T14-04-28-188/lre_avio_daq2.kicad_sch (KiCad schematic)
At the start: 150 parts, among them J1 Conn_01x02_Socket, J11 USB_C_Receptacle_USB2.0_16P, J12 XT30PW-F, J13 XT30PW-F, J14 XT30PW-F, J15 XT30PW-F, J16 XT30PW-F, J17 SMPW-CC-K-M, J18 SMPW-CC-K-M, J19 SMPW-CC-K-M, J2 DB25_Socket_MountingHoles, J23 DA15_Socket_MountingHoles, J24 DB25_Socket_MountingHoles, J3 XT60PW-M, Q1 SISA96DN-T1-GE3, Q2 SISA96DN-T1-GE3, Q3 SISA96DN-T1-GE3, SW1 SW_SPDT, U1 AMS1117-5.0, U10 ADS8353QPWRQ1, U11 ADS8353QPWRQ1, U12 STM32F412VGTx, U13 HX711, U14 HX711, U15 WS2812B-2020, U16 WS2812B-2020, U17 WS2812B-2020, U2 HX711, U3 SN65HVD230, U4 HX711, U5 AMS1117-5.0, U6 ADS8353QPWRQ1, U7 MAX31856, U8 MAX31856, U9 MAX31856, Y1 Crystal_8Mhz

Commit message: commit
Parts:
- removed D3: LED, LED_SMD:LED_0603_1608Metric, symbol Device:LED
- removed LS1: CMT-8530S-SMT, CMT-8530S-SMT:CUI_CMT-8530S-SMT, symbol CMT-8530S-SMT:CMT-8530S-SMT
- removed Q5: (no value), CJ3400:SOT95P240X115-3N, symbol CJ3400:CJ3400
- removed R34: R, Resistor_SMD:R_0603_1608Metric, symbol Device:R
- removed R35: 100, Resistor_SMD:R_0603_1608Metric, symbol Device:R_Small_US
- removed R36: 10k, Resistor_SMD:R_0603_1608Metric, symbol Device:R_Small_US
- removed U15, U16, U17: WS2812B-2020, SMT_12B-2020_WDS, symbol 2026-09-24_08-31-29:WS2812B-2020
Connections:
- net Buzzer_G: no longer names the net of U12.8 (PC14)
- net DI1: no longer names the net of U12.9 (PC15)
- no-connect marks 69 -> 70
